Commit message: Debugging path generation

File: avena_bringup/urdf/avena_arm_franka_hand.urdf.xacro (robot description, xacro)
@@ -3,4 +3,4 @@
   <xacro:include filename="$(find avena_bringup)/urdf/urdf_v4.urdf.xacro"/>
   <xacro:include filename="$(find avena_bringup)/urdf/hand.xacro"/>
-  <xacro:hand ns="panda" rpy="1 0 0" connected_to="Panda_gripper"/>
+  <xacro:hand ns="franka" rpy="1 0 0" connected_to="franka_gripper"/>
 </robot>

File: avena_bringup/urdf/calibration_mat.xacro (robot description, xacro)
@@ -3,5 +3,5 @@
   <!-- safety_distance: Minimum safety distance in [m] by which the collision volumes are expanded and which is enforced during robot motions -->
   <xacro:macro name="calibration_mat"
-               params="connected_to:='' grid_size:='1' description_pkg:='avena_bringup' arm_id:='panda' ns:='' rpy:='0 0 0' xyz:='0 0 0' safety_distance:=0">
+               params="connected_to:='' grid_size:='1' description_pkg:='avena_bringup' arm_id:='franka' ns:='' rpy:='0 0 0' xyz:='0 0 0' safety_distance:=0">
     <!-- ********************************************* -->
     <!-- Parameters -->

File: avena_bringup/urdf/franka.urdf.xacro (robot description, xacro)
@@ -1,9 +1,9 @@
 <?xml version="1.0" encoding="utf-8"?>
-<robot xmlns:xacro="http://www.ros.org/wiki/xacro" name="panda">
-  <xacro:include filename="$(find avena_bringup)/urdf/panda_arm.xacro"/>
+<robot xmlns:xacro="http://www.ros.org/wiki/xacro" name="franka">
+  <xacro:include filename="$(find avena_bringup)/urdf/franka_arm.xacro"/>
   <!-- <xacro:include filename="$(find avena_bringup)/urdf/hand.xacro"/> -->
   <xacro:arg name="side" default="right" />
   <xacro:arg name="description_pkg" default="avena_bringup" />
-  <xacro:panda_arm arm_id="$(arg side)_franka" description_pkg="$(arg description_pkg)" safety_distance="0.03"/>
+  <xacro:franka_arm arm_id="$(arg side)_franka" description_pkg="$(arg description_pkg)" safety_distance="0.03"/>
   <!-- <xacro:hand arm_id="$(arg side)_franka" rpy="0 0 ${-pi/4}" connected_to="$(arg side)_franka_gripper_connection" safety_distance="0.03"/> -->
 </robot>

File: avena_bringup/urdf/franka_calibration.urdf.xacro (robot description, xacro)
@@ -1,9 +1,9 @@
 <?xml version="1.0" encoding="utf-8"?>
-<robot xmlns:xacro="http://www.ros.org/wiki/xacro" name="panda">
-  <xacro:include filename="$(find avena_bringup)/urdf/panda_arm.xacro"/>
+<robot xmlns:xacro="http://www.ros.org/wiki/xacro" name="franka">
+  <xacro:include filename="$(find avena_bringup)/urdf/franka_arm.xacro"/>
   <xacro:include filename="$(find avena_bringup)/urdf/calibration_mat.xacro"/>
   <xacro:arg name="side" default="right" />
   <xacro:arg name="description_pkg" default="avena_bringup" />
-  <xacro:panda_arm arm_id="$(arg side)_franka" description_pkg="$(arg description_pkg)" safety_distance="0.03"/>
+  <xacro:franka_arm arm_id="$(arg side)_franka" description_pkg="$(arg description_pkg)" safety_distance="0.03"/>
   <!-- Calibration mat offsets -->
   <xacro:property name="grid_size" value="0.04025" />

File: avena_bringup/urdf/hand.urdf.xacro (robot description, xacro)
@@ -2,4 +2,4 @@
 <robot xmlns:xacro="http://www.ros.org/wiki/xacro" name="hand">
   <xacro:include filename="hand.xacro"/>
-  <xacro:hand ns="panda" safety_distance="0.03"/>
+  <xacro:hand ns="franka" safety_distance="0.03"/>
 </robot>

File: avena_bringup/urdf/hand.xacro (robot description, xacro)
@@ -2,5 +2,5 @@
 <robot xmlns:xacro="http://www.ros.org/wiki/xacro" name="hand">
   <!-- safety_distance: Minimum safety distance in [m] by which the collision volumes are expanded and which is enforced during robot motions -->
-  <xacro:macro name="hand" params="connected_to:=''  description_pkg:='avena_bringup' arm_id:='panda' ns:='' rpy:='0 0 0' xyz:='0 0 0' safety_distance:=0">
+  <xacro:macro name="hand" params="connected_to:=''  description_pkg:='avena_bringup' arm_id:='franka' ns:='' rpy:='0 0 0' xyz:='0 0 0' safety_distance:=0">
     <xacro:unless value="${connected_to == ''}">
       <joint name="${arm_id}_hand_joint" type="fixed">

File: avena_bringup/urdf/urdf_v4.urdf.xacro (robot description, xacro)
@@ -290,5 +290,5 @@
       velocity="0" />
   </joint>
-    <link name="Panda_gripper">
+    <link name="franka_gripper">
       <collision>
         <origin xyz="0 0 0" rpy="0 0 0"/>
@@ -313,5 +313,5 @@
       <origin rpy="-0.985 -1.57 2.55" xyz="0 -0.027 0"/>
       <parent link="left_link_6"/>
-      <child link="Panda_gripper"/>
+      <child link="franka_gripper"/>
     </joint>
 </robot>

File: avena_bringup/urdf/v4.urdf.xacro (robot description, xacro)
@@ -332,5 +332,5 @@
       velocity="0" />
   </joint>
-    <link name="Panda_gripper">
+    <link name="franka_gripper">
       <collision>
         <origin xyz="0 0 0" rpy="0 0 0"/>
@@ -360,5 +360,5 @@
       <origin rpy="-0.985 -1.57 2.55" xyz="0 -0.027 0"/>
       <parent link="left_link_6"/>
-      <child link="Panda_gripper"/>
+      <child link="franka_gripper"/>
     </joint> -->
 </robot>
