Commit message: It still does not work

File: avena_bringup/urdf/calibration_mat.xacro (robot description, xacro)
@@ -23,5 +23,5 @@
         <origin xyz="${1.5 * grid_size} ${grid_size} ${z_size/2}" rpy="0 0 0" />
         <geometry>
-          <box size="${x_size} ${y_size} ${z_size}" />
+          <box size="${x_size} ${y_size} ${z_size-0.01}" />
         </geometry>
         <material name="Grey">
@@ -32,5 +32,5 @@
         <origin xyz="${1.5 * grid_size} ${grid_size} ${z_size/2}" rpy="0 0 0" />
         <geometry>
-          <box size="${x_size} ${y_size} ${z_size}" />
+          <box size="${x_size} ${y_size} ${z_size-0.01}" />
         </geometry>
       </collision>

Commit message: Modify placement of calibration mat

File: avena_bringup/urdf/calibration_mat.xacro (robot description, xacro)
@@ -11,4 +11,5 @@
     <xacro:property name="y_size" value="0.17" />
     <xacro:property name="z_size" value="0.02306" />
+    <xacro:property name="z_offset" value="0.01" />
     <!-- ********************************************* -->
     <xacro:unless value="${connected_to == ''}">
@@ -21,7 +22,7 @@
     <link name="${arm_id}_calibration_mat">
       <visual>
-        <origin xyz="${1.5 * grid_size} ${grid_size} ${z_size/2}" rpy="0 0 0" />
+        <origin xyz="${1.5 * grid_size} ${grid_size} ${z_size/2-z_offset/2}" rpy="0 0 0" />
         <geometry>
-          <box size="${x_size} ${y_size} ${z_size-0.01}" />
+          <box size="${x_size} ${y_size} ${z_size-z_offset}" />
         </geometry>
         <material name="Grey">
@@ -30,7 +31,7 @@
       </visual>
       <collision>
-        <origin xyz="${1.5 * grid_size} ${grid_size} ${z_size/2}" rpy="0 0 0" />
+        <origin xyz="${1.5 * grid_size} ${grid_size} ${z_size/2-z_offset/2}" rpy="0 0 0" />
         <geometry>
-          <box size="${x_size} ${y_size} ${z_size-0.01}" />
+          <box size="${x_size} ${y_size} ${z_size-z_offset}" />
         </geometry>
       </collision>
