Commit message: controller with friction comp

File: avena_bringup/urdf/v4.urdf.xacro (robot description, xacro)
@@ -53,5 +53,5 @@
       lower="-3.05"
       upper="3.05"
-      effort="30."
+      effort="50."
       velocity="0." />
   </joint>
@@ -102,5 +102,5 @@
       lower="-1.57"
       upper="1.57"
-      effort="45."
+      effort="80."
       velocity="0." />
   </joint>
@@ -182,5 +182,5 @@
       lower="-2.9"
       upper="2.9"
-      effort="0"
+      effort="60."
       velocity="0" />
   </joint>
@@ -216,5 +216,14 @@
     </inertial>
   </link>
-  <joint
+  <joint name="dummy_joint" type="fixed">
+    <origin
+      xyz="0 0.447 0.0006"
+      rpy="1.5708 0 0" />
+    <parent
+      link="left_link_3" />
+    <child
+      link="left_link_4" />
+  </joint>
+  <!-- <joint
     name="left_joint_4"
     type="revolute">
@@ -282,5 +291,5 @@
       effort="0"
       velocity="0" />
-  </joint>
+  </joint> -->
   <!-- <link
     name="left_link_6">

Commit message: Revert "controller with friction comp"
This reverts commit 143c0c5a3b2aef22fe670d46ac10e3e82b76eea9.

File: avena_bringup/urdf/v4.urdf.xacro (robot description, xacro)
@@ -53,5 +53,5 @@
       lower="-3.05"
       upper="3.05"
-      effort="50."
+      effort="30."
       velocity="0." />
   </joint>
@@ -102,5 +102,5 @@
       lower="-1.57"
       upper="1.57"
-      effort="80."
+      effort="45."
       velocity="0." />
   </joint>
@@ -182,5 +182,5 @@
       lower="-2.9"
       upper="2.9"
-      effort="60."
+      effort="0"
       velocity="0" />
   </joint>
@@ -216,14 +216,5 @@
     </inertial>
   </link>
-  <joint name="dummy_joint" type="fixed">
-    <origin
-      xyz="0 0.447 0.0006"
-      rpy="1.5708 0 0" />
-    <parent
-      link="left_link_3" />
-    <child
-      link="left_link_4" />
-  </joint>
-  <!-- <joint
+  <joint
     name="left_joint_4"
     type="revolute">
@@ -291,5 +282,5 @@
       effort="0"
       velocity="0" />
-  </joint> -->
+  </joint>
   <!-- <link
     name="left_link_6">

Commit message: Revert "Revert "controller with friction comp"" duh
This reverts commit 24331205142ce974b9d2d13d26e46abc87577043.

File: avena_bringup/urdf/v4.urdf.xacro (robot description, xacro)
@@ -53,5 +53,5 @@
       lower="-3.05"
       upper="3.05"
-      effort="30."
+      effort="50."
       velocity="0." />
   </joint>
@@ -102,5 +102,5 @@
       lower="-1.57"
       upper="1.57"
-      effort="45."
+      effort="80."
       velocity="0." />
   </joint>
@@ -182,5 +182,5 @@
       lower="-2.9"
       upper="2.9"
-      effort="0"
+      effort="60."
       velocity="0" />
   </joint>
@@ -216,7 +216,5 @@
     </inertial>
   </link>
-  <joint
-    name="dummy"
-    type="fixed">
+  <joint name="dummy_joint" type="fixed">
     <origin
       xyz="0 0.447 0.0006"
@@ -343,5 +341,5 @@
       velocity="0" />
   </joint>
-    <link name="franka_gripper">
+    <link name="Panda_gripper">
       <collision>
         <origin xyz="0 0 0" rpy="0 0 0"/>
@@ -371,5 +369,5 @@
       <origin rpy="-0.985 -1.57 2.55" xyz="0 -0.027 0"/>
       <parent link="left_link_6"/>
-      <child link="franka_gripper"/>
+      <child link="Panda_gripper"/>
     </joint> -->
 </robot>
