Commit message: Run on Franka robot; working with IKFast

File: core/avena_bringup/urdf/calibration_mat.xacro (robot description, xacro)
@@ -24,5 +24,5 @@
         <origin xyz="${1.5 * grid_size} ${grid_size} ${z_size/2-z_offset/2}" rpy="0 0 0" />
         <geometry>
-          <box size="${x_size} ${y_size} ${z_size-z_offset}" />
+          <box size="${x_size + safety_distance} ${y_size + safety_distance} ${z_size-z_offset}" />
         </geometry>
         <material name="Grey">
@@ -33,5 +33,5 @@
         <origin xyz="${1.5 * grid_size} ${grid_size} ${z_size/2-z_offset/2}" rpy="0 0 0" />
         <geometry>
-          <box size="${x_size} ${y_size} ${z_size-z_offset}" />
+          <box size="${x_size + safety_distance} ${y_size + safety_distance} ${z_size-z_offset}" />
         </geometry>
       </collision>

File: core/avena_bringup/urdf/franka_arm.xacro (robot description, xacro)
@@ -4,11 +4,4 @@
   <!-- arm_id: Namespace of the franka arm. Serves to differentiate between arms in case of multiple instances. -->
   <xacro:macro name="franka_arm" params="arm_id:='franka' description_pkg:='avena_bringup' connected_to:='' xyz:='0 0 0' rpy:='0 0 0' safety_distance:=0">
-    <xacro:unless value="${not connected_to}">
-      <joint name="${arm_id}_joint__${connected_to}" type="fixed">
-        <parent link="${connected_to}"/>
-        <child link="${arm_id}_link_0"/>
-        <origin rpy="${rpy}" xyz="${xyz}"/>
-      </joint>
-    </xacro:unless>
     <link name="${arm_id}_link_0">
       <visual>
@@ -35,12 +28,4 @@
       </collision>
     </link>
-    <joint name="${arm_id}_joint_1" type="revolute">
-      <safety_controller k_position="100.0" k_velocity="40.0" soft_lower_limit="-2.8973" soft_upper_limit="2.8973"/>
-      <origin rpy="0 0 0" xyz="0 0 0.333"/>
-      <parent link="${arm_id}_link_0"/>
-      <child link="${arm_id}_link_1"/>
-      <axis xyz="0 0 1"/>
-      <limit effort="87" lower="-2.8973" upper="2.8973" velocity="2.1750"/>
-    </joint>
     <link name="${arm_id}_link_2">
       <visual>
@@ -55,12 +40,4 @@
       </collision>
     </link>
-    <joint name="${arm_id}_joint_2" type="revolute">
-      <safety_controller k_position="100.0" k_velocity="40.0" soft_lower_limit="-1.7628" soft_upper_limit="1.7628"/>
-      <origin rpy="${-pi/2} 0 0" xyz="0 0 0"/>
-      <parent link="${arm_id}_link_1"/>
-      <child link="${arm_id}_link_2"/>
-      <axis xyz="0 0 1"/>
-      <limit effort="87" lower="-1.7628" upper="1.7628" velocity="2.1750"/>
-    </joint>
     <link name="${arm_id}_link_3">
       <visual>
@@ -75,12 +52,4 @@
       </collision>
     </link>
-    <joint name="${arm_id}_joint_3" type="revolute">
-      <safety_controller k_position="100.0" k_velocity="40.0" soft_lower_limit="-2.8973" soft_upper_limit="2.8973"/>
-      <origin rpy="${pi/2} 0 0" xyz="0 -0.316 0"/>
-      <parent link="${arm_id}_link_2"/>
-      <child link="${arm_id}_link_3"/>
-      <axis xyz="0 0 1"/>
-      <limit effort="87" lower="-2.8973" upper="2.8973" velocity="2.1750"/>
-    </joint>
     <link name="${arm_id}_link_4">
       <visual>
@@ -95,12 +64,4 @@
       </collision>
     </link>
-    <joint name="${arm_id}_joint_4" type="revolute">
-      <safety_controller k_position="100.0" k_velocity="40.0" soft_lower_limit="-3.0718" soft_upper_limit="-0.0698"/>
-      <origin rpy="${pi/2} 0 0" xyz="0.0825 0 0"/>
-      <parent link="${arm_id}_link_3"/>
-      <child link="${arm_id}_link_4"/>
-      <axis xyz="0 0 1"/>
-      <limit effort="87" lower="-3.0718" upper="-0.0698" velocity="2.1750"/>
-    </joint>
     <link name="${arm_id}_link_5">
       <visual>
@@ -115,12 +76,4 @@
       </collision>
     </link>
-    <joint name="${arm_id}_joint_5" type="revolute">
-      <safety_controller k_position="100.0" k_velocity="40.0" soft_lower_limit="-2.8973" soft_upper_limit="2.8973"/>
-      <origin rpy="${-pi/2} 0 0" xyz="-0.0825 0.384 0"/>
-      <parent link="${arm_id}_link_4"/>
-      <child link="${arm_id}_link_5"/>
-      <axis xyz="0 0 1"/>
-      <limit effort="12" lower="-2.8973" upper="2.8973" velocity="2.6100"/>
-    </joint>
     <link name="${arm_id}_link_6">
       <visual>
@@ -135,12 +88,4 @@
       </collision>
     </link>
-    <joint name="${arm_id}_joint_6" type="revolute">
-      <safety_controller k_position="100.0" k_velocity="40.0" soft_lower_limit="-0.0175" soft_upper_limit="3.7525"/>
-      <origin rpy="${pi/2} 0 0" xyz="0 0 0"/>
-      <parent link="${arm_id}_link_5"/>
-      <child link="${arm_id}_link_6"/>
-      <axis xyz="0 0 1"/>
-      <limit effort="12" lower="-0.0175" upper="3.7525" velocity="2.6100"/>
-    </joint>
     <link name="${arm_id}_link_7">
       <visual>
@@ -155,4 +100,60 @@
       </collision>
     </link>
+    <link name="${arm_id}_gripper_connection"/>
+    <xacro:unless value="${not connected_to}">
+      <joint name="${arm_id}_joint__${connected_to}" type="fixed">
+        <parent link="${connected_to}"/>
+        <child link="${arm_id}_link_0"/>
+        <origin rpy="${rpy}" xyz="${xyz}"/>
+      </joint>
+    </xacro:unless>
+    <joint name="${arm_id}_joint_1" type="revolute">
+      <safety_controller k_position="100.0" k_velocity="40.0" soft_lower_limit="-2.8973" soft_upper_limit="2.8973"/>
+      <origin rpy="0 0 0" xyz="0 0 0.333"/>
+      <parent link="${arm_id}_link_0"/>
+      <child link="${arm_id}_link_1"/>
+      <axis xyz="0 0 1"/>
+      <limit effort="87" lower="-2.8973" upper="2.8973" velocity="2.1750"/>
+    </joint>
+    <joint name="${arm_id}_joint_2" type="revolute">
+      <safety_controller k_position="100.0" k_velocity="40.0" soft_lower_limit="-1.7628" soft_upper_limit="1.7628"/>
+      <origin rpy="${-pi/2} 0 0" xyz="0 0 0"/>
+      <parent link="${arm_id}_link_1"/>
+      <child link="${arm_id}_link_2"/>
+      <axis xyz="0 0 1"/>
+      <limit effort="87" lower="-1.7628" upper="1.7628" velocity="2.1750"/>
+    </joint>
+    <joint name="${arm_id}_joint_3" type="revolute">
+      <safety_controller k_position="100.0" k_velocity="40.0" soft_lower_limit="-2.8973" soft_upper_limit="2.8973"/>
+      <origin rpy="${pi/2} 0 0" xyz="0 -0.316 0"/>
+      <parent link="${arm_id}_link_2"/>
+      <child link="${arm_id}_link_3"/>
+      <axis xyz="0 0 1"/>
+      <limit effort="87" lower="-2.8973" upper="2.8973" velocity="2.1750"/>
+    </joint>
+    <joint name="${arm_id}_joint_4" type="revolute">
+      <safety_controller k_position="100.0" k_velocity="40.0" soft_lower_limit="-3.0718" soft_upper_limit="-0.0698"/>
+      <origin rpy="${pi/2} 0 0" xyz="0.0825 0 0"/>
+      <parent link="${arm_id}_link_3"/>
+      <child link="${arm_id}_link_4"/>
+      <axis xyz="0 0 1"/>
+      <limit effort="87" lower="-3.0718" upper="-0.0698" velocity="2.1750"/>
+    </joint>
+    <joint name="${arm_id}_joint_5" type="revolute">
+      <safety_controller k_position="100.0" k_velocity="40.0" soft_lower_limit="-2.8973" soft_upper_limit="2.8973"/>
+      <origin rpy="${-pi/2} 0 0" xyz="-0.0825 0.384 0"/>
+      <parent link="${arm_id}_link_4"/>
+      <child link="${arm_id}_link_5"/>
+      <axis xyz="0 0 1"/>
+      <limit effort="12" lower="-2.8973" upper="2.8973" velocity="2.6100"/>
+    </joint>
+    <joint name="${arm_id}_joint_6" type="revolute">
+      <safety_controller k_position="100.0" k_velocity="40.0" soft_lower_limit="-0.0175" soft_upper_limit="3.7525"/>
+      <origin rpy="${pi/2} 0 0" xyz="0 0 0"/>
+      <parent link="${arm_id}_link_5"/>
+      <child link="${arm_id}_link_6"/>
+      <axis xyz="0 0 1"/>
+      <limit effort="12" lower="-0.0175" upper="3.7525" velocity="2.6100"/>
+    </joint>
     <joint name="${arm_id}_joint_7" type="revolute">
       <safety_controller k_position="100.0" k_velocity="40.0" soft_lower_limit="-2.8973" soft_upper_limit="2.8973"/>
@@ -163,5 +164,4 @@
       <limit effort="12" lower="-2.8973" upper="2.8973" velocity="2.6100"/>
     </joint>
-    <link name="${arm_id}_gripper_connection"/>
     <joint name="${arm_id}_joint_8" type="fixed">
       <origin rpy="0 ${-pi/2} ${0.75*pi}" xyz="0 0 0.107"/>
