Commit message: Update reading robot info from URDF

File: core/avena_bringup/urdf/franka.urdf.xacro (robot description, xacro)
@@ -2,8 +2,8 @@
 <robot xmlns:xacro="http://www.ros.org/wiki/xacro" name="franka">
   <xacro:include filename="$(find avena_bringup)/urdf/franka_arm.xacro"/>
-  <!-- <xacro:include filename="$(find avena_bringup)/urdf/hand.xacro"/> -->
+  <xacro:include filename="$(find avena_bringup)/urdf/hand.xacro"/>
   <xacro:arg name="side" default="right" />
   <xacro:arg name="description_pkg" default="avena_bringup" />
   <xacro:franka_arm arm_id="$(arg side)_franka" description_pkg="$(arg description_pkg)" safety_distance="0.03"/>
-  <!-- <xacro:hand arm_id="$(arg side)_franka" rpy="0 0 ${-pi/4}" connected_to="$(arg side)_franka_gripper_connection" safety_distance="0.03"/> -->
+  <xacro:hand arm_id="$(arg side)_franka" rpy="${pi} ${-pi/2} 0" connected_to="$(arg side)_franka_gripper_connection" safety_distance="0.03"/>
 </robot>

File: core/avena_bringup/urdf/hand.xacro (robot description, xacro)
@@ -7,5 +7,5 @@
         <parent link="${connected_to}"/>
         <child link="${arm_id}_gripper"/>
-        <origin xyz="${xyz}" rpy="0 0 -0.785"/>
+        <origin xyz="${xyz}" rpy="${rpy}"/>
       </joint>
     </xacro:unless>

Commit message: Change end effector approach vector and update _rotateSamples in camera...

File: core/avena_bringup/urdf/franka.urdf.xacro (robot description, xacro)
@@ -6,4 +6,4 @@
   <xacro:arg name="description_pkg" default="avena_bringup" />
   <xacro:franka_arm arm_id="$(arg side)_franka" description_pkg="$(arg description_pkg)" safety_distance="0.03"/>
-  <xacro:hand arm_id="$(arg side)_franka" rpy="${pi} ${-pi/2} 0" connected_to="$(arg side)_franka_gripper_connection" safety_distance="0.03"/>
+  <xacro:hand arm_id="$(arg side)_franka" rpy="0 0 0" connected_to="$(arg side)_franka_gripper_connection" safety_distance="0.03"/>
 </robot>

File: core/avena_bringup/urdf/franka_arm.xacro (robot description, xacro)
@@ -167,7 +167,8 @@
     </joint>
     <joint name="${arm_id}_joint_8" type="fixed">
-      <origin rpy="0 ${-pi/2} ${0.75*pi}" xyz="0 0 0.107"/>
+      <origin rpy="0 0 ${-pi/4}" xyz="0 0 0.107"/>
       <parent link="${arm_id}_link_7"/>
       <child link="${arm_id}_gripper_connection"/>
+      <axis xyz="0 0 0"/>
     </joint>
   </xacro:macro>

File: core/avena_bringup/urdf/franka_calibration.urdf.xacro (robot description, xacro)
@@ -8,10 +8,10 @@
   <!-- Calibration mat offsets -->
   <xacro:property name="grid_size" value="0.04025" />
-  <xacro:property name="x_axis_offset" value="0.02306" />
-  <xacro:property name="y_axis_offset" value="${-1.5 * grid_size}" />
-  <xacro:property name="z_axis_offset" value="${grid_size}" />
-  <xacro:property name="x_axis_rot" value="${-pi/2}" />
+  <xacro:property name="x_axis_offset" value="${grid_size}" />
+  <xacro:property name="y_axis_offset" value="${1.5 * grid_size}" />
+  <xacro:property name="z_axis_offset" value="0.02306" />
+  <xacro:property name="x_axis_rot" value="${pi}" />
   <xacro:property name="y_axis_rot" value="0" />
-  <xacro:property name="z_axis_rot" value="${pi/2}" />
+  <xacro:property name="z_axis_rot" value="${-pi/2}" />
   <xacro:calibration_mat arm_id="$(arg side)_franka"
                          connected_to="$(arg side)_franka_gripper_connection"
