Commit message: config update

File: core/avena_bringup/urdf/avena_arm_old.xacro (robot description, xacro)
@@ -49,5 +49,5 @@
     <link name="${arm_id}_link_2">
       <visual>
-        <origin xyz="0 0 0.0" rpy="0 ${pi} ${pi/2}" />
+        <origin xyz="0 0 0.0763" rpy="0 ${pi} ${pi/2}" />
         <geometry>
           <mesh filename="file://$(find ${description_pkg})/urdf/meshes/avena/link_2.stl" scale="0.001 0.001 0.001" />
@@ -56,10 +56,10 @@
       </visual>
       <inertial>
-        <origin xyz="-0.343 0. 0.05884" rpy="0. ${pi} ${pi/2}"/>
+        <origin xyz="-0.17651 0. 0.01528" rpy="0. ${pi} ${pi/2}"/>
         <mass value="9."/>
-        <inertia ixx="8.437e-01"  ixy="0."  ixz="0." iyy="1.143e-02" iyz="0." izz="8.428e-01" />
-      </inertial>
-      <collision>
-        <origin xyz="0 0 0" rpy="0 ${pi} ${pi/2}" />
+        <inertia ixx="2.809e-01"  ixy="0."  ixz="0." iyy="8.463e-03" iyz="0." izz="2.804e-01" />
+      </inertial>
+      <collision>
+        <origin xyz="0 0 0.0763" rpy="0 ${pi} ${pi/2}" />
         <geometry>
           <mesh filename="file://$(find ${description_pkg})/urdf/meshes/avena/link_2.stl" scale="0.001 0.001 0.001" />
@@ -69,5 +69,5 @@
     <link name="${arm_id}_link_3">
       <visual>
-        <origin xyz="0. 0. 0.0" rpy="0 ${pi} ${-pi/2}" />
+        <origin xyz="0. 0. 0.0721" rpy="0 ${pi} ${-pi/2}" />
         <geometry>
           <mesh filename="file://$(find ${description_pkg})/urdf/meshes/avena/link_3.stl" scale="0.001 0.001 0.001" />
@@ -76,10 +76,10 @@
       </visual>
       <inertial>
-        <origin xyz="0.38666 0. 0.051" rpy="0 0 ${pi/2}"/>
-        <mass value="5."/>
-        <inertia ixx="3.605e-01"  ixy="0"  ixz="0" iyy="6.825e-03" iyz="0" izz="3.606e-01" />
-      </inertial>
-      <collision>
-        <origin xyz="0 0 0" rpy="0 ${pi} ${-pi/2}" />
+        <origin xyz="0.3046 0. 0.0588" rpy="0 0 ${pi/2}"/>
+        <mass value="3.375"/>
+        <inertia ixx="1.149e-01"  ixy="0"  ixz="0" iyy="4.518e-03" iyz="0" izz="1.148e-01" />
+      </inertial>
+      <collision>
+        <origin xyz="0 0 0.0721" rpy="0 ${pi} ${-pi/2}" />
         <geometry>
           <mesh filename="file://$(find ${description_pkg})/urdf/meshes/avena/link_3.stl" scale="0.001 0.001 0.001" />
@@ -97,5 +97,5 @@
       <inertial>
         <origin xyz="0.019 0. 0.059 " rpy="0. 0. ${pi/2}"/>
-        <mass value="2."/>
+        <mass value="1.960"/>
         <inertia ixx="2.233e-03"  ixy="0."  ixz="0." iyy="2.047e-03" iyz="0." izz="2.384e-03" />
       </inertial>
@@ -117,5 +117,5 @@
       <inertial>
         <origin xyz="0.019 0 0.059" rpy="0. 0. ${pi/2}"/>
-        <mass value="2."/>
+        <mass value="1.960"/>
         <inertia ixx="2.233e-03"  ixy="0."  ixz="0." iyy="2.047e-03" iyz="0." izz="2.384e-03" />
       </inertial>
@@ -156,9 +156,9 @@
     </joint>
     <joint name="${arm_id}_joint_1" type="revolute">
-      <origin xyz="0 0 0.063" rpy="0 0 0" /> <!-- Offset from position -->
+      <origin xyz="0 0 0.063" rpy="0 0 -0.1963" /> <!-- Offset from position -->
       <parent link="${arm_id}_link_0" />
       <child link="${arm_id}_link_1" />
       <axis xyz="0 0 1" />
-      <limit lower="-3.05" upper="3.05" effort="80" velocity="1." />
+      <limit lower="-3.05" upper="3.05" effort="80" velocity="0" />
     </joint>
     <joint name="${arm_id}_joint_2" type="revolute">
@@ -167,19 +167,19 @@
       <child link="${arm_id}_link_2" />
       <axis xyz="0 0 1" />
-      <limit lower="-1.57" upper="1.57" effort="250" velocity="1." />
+      <limit lower="-1.57" upper="1.57" effort="180" velocity="0" />
     </joint>
     <joint name="${arm_id}_joint_3" type="revolute">
-      <origin xyz="-0.686 0 0" rpy="0 ${pi} 0" />
+      <origin xyz="-0.467 0 0.009" rpy="0 ${pi} 0" />
       <parent link="${arm_id}_link_2" />
       <child link="${arm_id}_link_3" />
       <axis xyz="0 0 1" />
-      <limit lower="-2.9" upper="2.9" effort="120" velocity="1." />
+      <limit lower="-2.9" upper="2.9" effort="120" velocity="0" />
     </joint>
     <joint name="${arm_id}_joint_4" type="revolute">
-      <origin xyz="0.671 0 -0.005" rpy="${pi} 0 0" />
+      <origin xyz="0.452 0 0.0226" rpy="${pi} 0 0" />
       <parent link="${arm_id}_link_3" />
       <child link="${arm_id}_link_4" />
       <axis xyz="0 0 1" />
-      <limit lower="-3.05" upper="3.05" effort="60" velocity="1." />
+      <limit lower="-3.05" upper="3.05" effort="60" velocity="0" />
     </joint>
     <joint name="${arm_id}_joint_5" type="revolute">
@@ -188,5 +188,5 @@
       <child link="${arm_id}_link_5" />
       <axis xyz="0 0 1" />
-      <limit lower="-3.05" upper="3.05" effort="40" velocity="1." />
+      <limit lower="-3.05" upper="3.05" effort="40" velocity="0" />
     </joint>
     <joint name="${arm_id}_joint_6" type="revolute">
@@ -195,5 +195,5 @@
       <child link="${arm_id}_link_6" />
       <axis xyz="0 0 1" />
-      <limit lower="-3.05" upper="3.05" effort="40" velocity="1." />
+      <limit lower="-3.05" upper="3.05" effort="40" velocity="0" />
     </joint>
     <joint name="${arm_id}_joint_7" type="fixed">
