Commit message: Modified avena arm URDF to have xacro macros to modify prefix; organize URDF file

File: core/avena_bringup/urdf/avena_arm.xacro (robot description, xacro)
@@ -1,189 +1,192 @@
 <?xml version="1.0" encoding="utf-8"?>
 <robot xmlns:xacro="http://www.ros.org/wiki/xacro" name="avena">
-  <link name="left_avena_link_0">
-    <visual>
-      <origin xyz="0 0 0" rpy="0 0 0" />
-      <geometry>
-        <mesh filename="package://avena_bringup/urdf/meshes/base_link.stl" />
-      </geometry>
-      <material name="">
-        <color rgba="0.898039215686275 0.917647058823529 0.929411764705882 1" />
-      </material>
-    </visual>
-    <collision>
-      <origin xyz="0 0 0" rpy="0 0 0" />
-      <geometry>
-        <mesh filename="package://avena_bringup/urdf/meshes/base_link.stl" />
-      </geometry>
-    </collision>
-  </link>
-  <link name="left_avena_link_1">
-    <visual>
-      <origin xyz="0 0 0" rpy="0 0 0" />
-      <geometry>
-        <mesh filename="package://avena_bringup/urdf/meshes/Link_1.stl" />
-      </geometry>
-      <material name="">
-        <color rgba="0.752941176470588 0.752941176470588 0.752941176470588 1" />
-      </material>
-    </visual>
-    <collision>
-      <origin xyz="0 0 0" rpy="0 0 0" />
-      <geometry>
-        <mesh filename="package://avena_bringup/urdf/meshes/Link_1.stl" />
-      </geometry>
-    </collision>
-  </link>
-  <joint name="left_avena_joint_1" type="revolute">
-    <origin xyz="0 0 0.047" rpy="3.1416 0 1.5708" />
-    <parent link="left_avena_link_0" />
-    <child link="left_avena_link_1" />
-    <axis xyz="0 0 -1" />
-    <limit lower="-3.05" upper="3.05" effort="0" velocity="0" />
-  </joint>
-  <link name="left_avena_link_2">
-    <visual>
-      <origin xyz="0 0 0" rpy="0 0 0" />
-      <geometry>
-        <mesh filename="package://avena_bringup/urdf/meshes/Link_2.stl" />
-      </geometry>
-      <material name="">
-        <color rgba="0.752941176470588 0.752941176470588 0.752941176470588 1" />
-      </material>
-    </visual>
-    <collision>
-      <origin xyz="0 0 0" rpy="0 0 0" />
-      <geometry>
-        <mesh filename="package://avena_bringup/urdf/meshes/Link_2.stl" />
-      </geometry>
-    </collision>
-  </link>
-  <joint name="left_avena_joint_2" type="revolute">
-    <origin xyz="0 0.048 -0.0679" rpy="-1.5708 0 0" />
-    <parent link="left_avena_link_1" />
-    <child link="left_avena_link_2" />
-    <axis xyz="0 0 1" />
-    <limit lower="-1.57" upper="1.57" effort="0" velocity="0" />
-  </joint>
-  <link name="left_avena_link_3">
-    <visual>
-      <origin xyz="0 0 0" rpy="0 0 0" />
-      <geometry>
-        <mesh filename="package://avena_bringup/urdf/meshes/Link_3.stl" />
-      </geometry>
-      <material name="">
-        <color rgba="0.752941176470588 0.752941176470588 0.752941176470588 1" />
-      </material>
-    </visual>
-    <collision>
-      <origin xyz="0 0 0" rpy="0 0 0" />
-      <geometry>
-        <mesh filename="package://avena_bringup/urdf/meshes/Link_3.stl" />
-      </geometry>
-    </collision>
-  </link>
-  <joint name="left_avena_joint_3" type="revolute">
-    <origin xyz="0 0.452 0" rpy="0 0 0" />
-    <parent link="left_avena_link_2" />
-    <child link="left_avena_link_3" />
-    <axis xyz="0 0 1" />
-    <limit lower="-2.9" upper="2.9" effort="0" velocity="0" />
-  </joint>
-  <link name="left_avena_link_4">
-    <visual>
-      <origin xyz="0 0 0" rpy="0 0 0" />
-      <geometry>
-        <mesh filename="package://avena_bringup/urdf/meshes/Link_4.stl" />
-      </geometry>
-      <material name="">
-        <color rgba="0.898039215686275 0.917647058823529 0.929411764705882 1" />
-      </material>
-    </visual>
-    <collision>
-      <origin xyz="0 0 0" rpy="0 0 0" />
-      <geometry>
-        <mesh filename="package://avena_bringup/urdf/meshes/Link_4.stl" />
-      </geometry>
-    </collision>
-  </link>
-  <joint name="left_avena_joint_4" type="revolute">
-    <origin xyz="0 0.447 0.0006" rpy="1.5708 0 0" />
-    <parent link="left_avena_link_3" />
-    <child link="left_avena_link_4" />
-    <axis xyz="0 1 0" />
-    <limit lower="-3.05" upper="3.05" effort="0" velocity="0" />
-  </joint>
-  <link name="left_avena_link_5">
-    <visual>
-      <origin xyz="0 0 0" rpy="0 0 0" />
-      <geometry>
-        <mesh filename="package://avena_bringup/urdf/meshes/Link_5.stl" />
-      </geometry>
-      <material name="">
-        <color rgba="0.898039215686275 0.917647058823529 0.929411764705882 1" />
-      </material>
-    </visual>
-    <collision>
-      <origin xyz="0 0 0" rpy="0 0 0" />
-      <geometry>
-        <mesh filename="package://avena_bringup/urdf/meshes/Link_5.stl" />
-      </geometry>
-    </collision>
-  </link>
-  <joint name="left_avena_joint_5" type="revolute">
-    <origin xyz="0 0.055 -0.0567" rpy="1.5708 0 3.1416" />
-    <parent link="left_avena_link_4" />
-    <child link="left_avena_link_5" />
-    <axis xyz="0 -1 0" />
-    <limit lower="-3.05" upper="3.05" effort="0" velocity="0" />
-  </joint>
-  <link name="left_avena_link_6">
-    <visual>
-      <origin xyz="0 0 0" rpy="0 0 0" />
-      <geometry>
-        <mesh filename="package://avena_bringup/urdf/meshes/Link_6.stl" />
-      </geometry>
-      <material name="">
-        <color rgba="0.898039215686275 0.917647058823529 0.929411764705882 1" />
-      </material>
-    </visual>
-    <collision>
-      <origin xyz="0 0 0" rpy="0 0 0" />
-      <geometry>
-        <mesh filename="package://avena_bringup/urdf/meshes/Link_6.stl" />
-      </geometry>
-    </collision>
-  </link>
-  <joint name="left_avena_joint_6" type="revolute">
-    <origin xyz="0 -0.055 0.0567" rpy="-1.5708 0 0.785" />
-    <parent link="left_avena_link_5" />
-    <child link="left_avena_link_6" />
-    <axis xyz="0 -1 0" />
-    <limit lower="-3.05" upper="3.05" effort="0" velocity="0" />
-  </joint>
-  <link name="franka_gripper">
-    <collision>
-      <origin xyz="0 0 0" rpy="0 0 0" />
-      <geometry>
-        <cylinder radius="0.03" length="0.01" />
-      </geometry>
-    </collision>
-    <collision>
-      <origin xyz="0.0424 0.0424 -0.02" rpy="0 0 0" />
-      <geometry>
-        <sphere radius="0.03" />
-      </geometry>
-    </collision>
-    <collision>
-      <origin xyz="0.0424 0.0424 -0.03" rpy="0 0 0" />
-      <geometry>
-        <sphere radius="0.03" />
-      </geometry>
-    </collision>
-  </link>
-  <joint name="left_avena_joint_7" type="fixed">
-    <origin rpy="-0.985 -1.57 2.55" xyz="0 -0.027 0" />
-    <parent link="left_avena_link_6" />
-    <child link="franka_gripper" />
-  </joint>
+  <xacro:macro name="avena_arm" params="arm_id:='avena' description_pkg:='avena_bringup'">
+    <link name="${arm_id}_link_0">
+      <visual>
+        <origin xyz="0 0 0" rpy="0 0 0" />
+        <geometry>
+          <mesh filename="file://$(find ${description_pkg})/urdf/meshes/base_link.stl" />
+        </geometry>
+        <material name="">
+          <color rgba="0.898039215686275 0.917647058823529 0.929411764705882 1" />
+        </material>
+      </visual>
+      <collision>
+        <origin xyz="0 0 0" rpy="0 0 0" />
+        <geometry>
+          <mesh filename="file://$(find ${description_pkg})/urdf/meshes/base_link.stl" />
+        </geometry>
+      </collision>
+    </link>
+    <link name="${arm_id}_link_1">
+      <visual>
+        <origin xyz="0 0 0" rpy="0 0 0" />
+        <geometry>
+          <mesh filename="file://$(find ${description_pkg})/urdf/meshes/Link_1.stl" />
+        </geometry>
+        <material name="">
+          <color rgba="0.752941176470588 0.752941176470588 0.752941176470588 1" />
+        </material>
+      </visual>
+      <collision>
+        <origin xyz="0 0 0" rpy="0 0 0" />
+        <geometry>
+          <mesh filename="file://$(find ${description_pkg})/urdf/meshes/Link_1.stl" />
+        </geometry>
+      </collision>
+    </link>
+    <link name="${arm_id}_link_2">
+      <visual>
+        <origin xyz="0 0 0" rpy="0 0 0" />
+        <geometry>
+          <mesh filename="file://$(find ${description_pkg})/urdf/meshes/Link_2.stl" />
+        </geometry>
+        <material name="">
+          <color rgba="0.752941176470588 0.752941176470588 0.752941176470588 1" />
+        </material>
+      </visual>
+      <collision>
+        <origin xyz="0 0 0" rpy="0 0 0" />
+        <geometry>
+          <mesh filename="file://$(find ${description_pkg})/urdf/meshes/Link_2.stl" />
+        </geometry>
+      </collision>
+    </link>
+    <link name="${arm_id}_link_3">
+      <visual>
+        <origin xyz="0 0 0" rpy="0 0 0" />
+        <geometry>
+          <mesh filename="file://$(find ${description_pkg})/urdf/meshes/Link_3.stl" />
+        </geometry>
+        <material name="">
+          <color rgba="0.752941176470588 0.752941176470588 0.752941176470588 1" />
+        </material>
+      </visual>
+      <collision>
+        <origin xyz="0 0 0" rpy="0 0 0" />
+        <geometry>
+          <mesh filename="file://$(find ${description_pkg})/urdf/meshes/Link_3.stl" />
+        </geometry>
+      </collision>
+    </link>
+    <link name="${arm_id}_link_4">
+      <visual>
+        <origin xyz="0 0 0" rpy="0 0 0" />
+        <geometry>
+          <mesh filename="file://$(find ${description_pkg})/urdf/meshes/Link_4.stl" />
+        </geometry>
+        <material name="">
+          <color rgba="0.898039215686275 0.917647058823529 0.929411764705882 1" />
+        </material>
+      </visual>
+      <collision>
+        <origin xyz="0 0 0" rpy="0 0 0" />
+        <geometry>
+          <mesh filename="file://$(find ${description_pkg})/urdf/meshes/Link_4.stl" />
+        </geometry>
+      </collision>
+    </link>
+    <link name="${arm_id}_link_5">
+      <visual>
+        <origin xyz="0 0 0" rpy="0 0 0" />
+        <geometry>
+          <mesh filename="file://$(find ${description_pkg})/urdf/meshes/Link_5.stl" />
+        </geometry>
+        <material name="">
+          <color rgba="0.898039215686275 0.917647058823529 0.929411764705882 1" />
+        </material>
+      </visual>
+      <collision>
+        <origin xyz="0 0 0" rpy="0 0 0" />
+        <geometry>
+          <mesh filename="file://$(find ${description_pkg})/urdf/meshes/Link_5.stl" />
+        </geometry>
+      </collision>
+    </link>
+    <link name="${arm_id}_link_6">
+      <visual>
+        <origin xyz="0 0 0" rpy="0 0 0" />
+        <geometry>
+          <mesh filename="file://$(find ${description_pkg})/urdf/meshes/Link_6.stl" />
+        </geometry>
+        <material name="">
+          <color rgba="0.898039215686275 0.917647058823529 0.929411764705882 1" />
+        </material>
+      </visual>
+      <collision>
+        <origin xyz="0 0 0" rpy="0 0 0" />
+        <geometry>
+          <mesh filename="file://$(find ${description_pkg})/urdf/meshes/Link_6.stl" />
+        </geometry>
+      </collision>
+    </link>
+    <!-- Joints -->
+    <joint name="${arm_id}_joint_1" type="revolute">
+      <origin xyz="0 0 0.047" rpy="3.1416 0 1.5708" />
+      <parent link="${arm_id}_link_0" />
+      <child link="${arm_id}_link_1" />
+      <axis xyz="0 0 -1" />
+      <limit lower="-3.05" upper="3.05" effort="0" velocity="0" />
+    </joint>
+    <joint name="${arm_id}_joint_2" type="revolute">
+      <origin xyz="0 0.048 -0.0679" rpy="-1.5708 0 0" />
+      <parent link="${arm_id}_link_1" />
+      <child link="${arm_id}_link_2" />
+      <axis xyz="0 0 1" />
+      <limit lower="-1.57" upper="1.57" effort="0" velocity="0" />
+    </joint>
+    <joint name="${arm_id}_joint_3" type="revolute">
+      <origin xyz="0 0.452 0" rpy="0 0 0" />
+      <parent link="${arm_id}_link_2" />
+      <child link="${arm_id}_link_3" />
+      <axis xyz="0 0 1" />
+      <limit lower="-2.9" upper="2.9" effort="0" velocity="0" />
+    </joint>
+    <joint name="${arm_id}_joint_4" type="revolute">
+      <origin xyz="0 0.447 0.0006" rpy="1.5708 0 0" />
+      <parent link="${arm_id}_link_3" />
+      <child link="${arm_id}_link_4" />
+      <axis xyz="0 1 0" />
+      <limit lower="-3.05" upper="3.05" effort="0" velocity="0" />
+    </joint>
+    <joint name="${arm_id}_joint_5" type="revolute">
+      <origin xyz="0 0.055 -0.0567" rpy="1.5708 0 3.1416" />
+      <parent link="${arm_id}_link_4" />
+      <child link="${arm_id}_link_5" />
+      <axis xyz="0 -1 0" />
+      <limit lower="-3.05" upper="3.05" effort="0" velocity="0" />
+    </joint>
+    <joint name="${arm_id}_joint_6" type="revolute">
+      <origin xyz="0 -0.055 0.0567" rpy="-1.5708 0 0.785" />
+      <parent link="${arm_id}_link_5" />
+      <child link="${arm_id}_link_6" />
+      <axis xyz="0 -1 0" />
+      <limit lower="-3.05" upper="3.05" effort="0" velocity="0" />
+    </joint>
+    <!--link name="franka_gripper">
+      <collision>
+        <origin xyz="0 0 0" rpy="0 0 0" />
+        <geometry>
+          <cylinder radius="0.03" length="0.01" />
+        </geometry>
+      </collision>
+      <collision>
+        <origin xyz="0.0424 0.0424 -0.02" rpy="0 0 0" />
+        <geometry>
+          <sphere radius="0.03" />
+        </geometry>
+      </collision>
+      <collision>
+        <origin xyz="0.0424 0.0424 -0.03" rpy="0 0 0" />
+        <geometry>
+          <sphere radius="0.03" />
+        </geometry>
+      </collision>
+    </link>
+    <joint name="${arm_id}_joint_7" type="fixed">
+      <origin rpy="-0.985 -1.57 2.55" xyz="0 -0.027 0" />
+      <parent link="${arm_id}_link_6" />
+      <child link="franka_gripper" />
+    </joint-->
+ </xacro:macro>
 </robot>

File: core/avena_bringup/urdf/avena_calibration.urdf.xacro (robot description, xacro)
@@ -2,10 +2,10 @@
 <robot xmlns:xacro="http://www.ros.org/wiki/xacro" name="avena">
   <xacro:include filename="$(find avena_bringup)/urdf/avena_arm.xacro"/>
-  <xacro:include filename="$(find avena_bringup)/urdf/calibration_mat.xacro"/>
+  <!-- <xacro:include filename="$(find avena_bringup)/urdf/calibration_mat.xacro"/> -->
   <xacro:arg name="side" default="right" />
   <xacro:arg name="description_pkg" default="avena_bringup" />
-  <xacro:franka_arm arm_id="$(arg side)_franka" description_pkg="$(arg description_pkg)" safety_distance="0.03"/>
+  <xacro:avena_arm arm_id="$(arg side)_avena" description_pkg="$(arg description_pkg)"/>
   <!-- Calibration mat offsets -->
-  <xacro:property name="grid_size" value="0.04025" />
+  <!-- <xacro:property name="grid_size" value="0.04025" />
   <xacro:property name="x_axis_offset" value="0.02306" />
   <xacro:property name="y_axis_offset" value="${-1.5 * grid_size}" />
@@ -19,4 +19,4 @@
                          xyz="${x_axis_offset} ${y_axis_offset} ${z_axis_offset}"
                          rpy="${x_axis_rot} ${y_axis_rot} ${z_axis_rot}"
-                         safety_distance="0.03"/>
+                         safety_distance="0.03"/> -->
 </robot>

Commit message: Spawning Avena arm in Bullet physics server; add gripper_connection joint

File: core/avena_bringup/urdf/avena_arm.xacro (robot description, xacro)
@@ -121,4 +121,5 @@
       </collision>
     </link>
+    <link name="${arm_id}_gripper_connection"/>
     <!-- Joints -->
     <joint name="${arm_id}_joint_1" type="revolute">
@@ -164,4 +165,9 @@
       <limit lower="-3.05" upper="3.05" effort="0" velocity="0" />
     </joint>
+    <joint name="${arm_id}_joint_7" type="fixed">
+      <origin rpy="0 0 0" xyz="0 -0.018 0"/>
+      <parent link="${arm_id}_link_6"/>
+      <child link="${arm_id}_gripper_connection"/>
+    </joint>
     <!--link name="franka_gripper">
       <collision>

File: core/avena_bringup/urdf/franka_arm.xacro (robot description, xacro)
@@ -4,5 +4,6 @@
   <!-- arm_id: Namespace of the franka arm. Serves to differentiate between arms in case of multiple instances. -->
   <xacro:macro name="franka_arm" params="arm_id:='franka' description_pkg:='avena_bringup' connected_to:='' xyz:='0 0 0' rpy:='0 0 0' safety_distance:=0">
-    <link name="${arm_id}_link_0">
+  <!-- Links   -->
+  <link name="${arm_id}_link_0">
       <visual>
         <geometry>
@@ -101,4 +102,5 @@
     </link>
     <link name="${arm_id}_gripper_connection"/>
+    <!-- Joints -->
     <xacro:unless value="${not connected_to}">
       <joint name="${arm_id}_joint__${connected_to}" type="fixed">

Commit message: Working IK fast for Avena arm

File: core/avena_bringup/urdf/avena_arm.xacro (robot description, xacro)
@@ -72,5 +72,5 @@
     <link name="${arm_id}_link_4">
       <visual>
-        <origin xyz="0 0 0" rpy="0 0 0" />
+        <origin xyz="0 0 0" rpy="${pi/2} 0 0" />
         <geometry>
           <mesh filename="file://$(find ${description_pkg})/urdf/meshes/Link_4.stl" />
@@ -81,5 +81,5 @@
       </visual>
       <collision>
-        <origin xyz="0 0 0" rpy="0 0 0" />
+        <origin xyz="0 0 0" rpy="${pi/2} 0 0" />
         <geometry>
           <mesh filename="file://$(find ${description_pkg})/urdf/meshes/Link_4.stl" />
@@ -89,5 +89,5 @@
     <link name="${arm_id}_link_5">
       <visual>
-        <origin xyz="0 0 0" rpy="0 0 0" />
+        <origin xyz="0 0 0" rpy="${-pi/2} 0 0" />
         <geometry>
           <mesh filename="file://$(find ${description_pkg})/urdf/meshes/Link_5.stl" />
@@ -98,5 +98,5 @@
       </visual>
       <collision>
-        <origin xyz="0 0 0" rpy="0 0 0" />
+        <origin xyz="0 0 0" rpy="${-pi/2} 0 0" />
         <geometry>
           <mesh filename="file://$(find ${description_pkg})/urdf/meshes/Link_5.stl" />
@@ -106,5 +106,5 @@
     <link name="${arm_id}_link_6">
       <visual>
-        <origin xyz="0 0 0" rpy="0 0 0" />
+        <origin xyz="0 0 0" rpy="${-pi/2} 0 0" />
         <geometry>
           <mesh filename="file://$(find ${description_pkg})/urdf/meshes/Link_6.stl" />
@@ -115,5 +115,5 @@
       </visual>
       <collision>
-        <origin xyz="0 0 0" rpy="0 0 0" />
+        <origin xyz="0 0 0" rpy="${-pi/2} 0 0" />
         <geometry>
           <mesh filename="file://$(find ${description_pkg})/urdf/meshes/Link_6.stl" />
@@ -124,12 +124,12 @@
     <!-- Joints -->
     <joint name="${arm_id}_joint_1" type="revolute">
-      <origin xyz="0 0 0.047" rpy="3.1416 0 1.5708" />
+      <origin xyz="0 0 0.047" rpy="${pi} 0 ${pi/2}" />
       <parent link="${arm_id}_link_0" />
       <child link="${arm_id}_link_1" />
-      <axis xyz="0 0 -1" />
+      <axis xyz="0 0 1" />
       <limit lower="-3.05" upper="3.05" effort="0" velocity="0" />
     </joint>
     <joint name="${arm_id}_joint_2" type="revolute">
-      <origin xyz="0 0.048 -0.0679" rpy="-1.5708 0 0" />
+      <origin xyz="0 0.048 -0.0679" rpy="-${pi/2} 0 0" />
       <parent link="${arm_id}_link_1" />
       <child link="${arm_id}_link_2" />
@@ -145,54 +145,30 @@
     </joint>
     <joint name="${arm_id}_joint_4" type="revolute">
-      <origin xyz="0 0.447 0.0006" rpy="1.5708 0 0" />
+      <origin xyz="0 0.447 0.0006" rpy="0 0 0" />
       <parent link="${arm_id}_link_3" />
       <child link="${arm_id}_link_4" />
-      <axis xyz="0 1 0" />
+      <axis xyz="0 0 1" />
       <limit lower="-3.05" upper="3.05" effort="0" velocity="0" />
     </joint>
     <joint name="${arm_id}_joint_5" type="revolute">
-      <origin xyz="0 0.055 -0.0567" rpy="1.5708 0 3.1416" />
+      <origin xyz="0 0.0567 0.055" rpy="${pi/2} 0 ${pi}" />
       <parent link="${arm_id}_link_4" />
       <child link="${arm_id}_link_5" />
-      <axis xyz="0 -1 0" />
+      <axis xyz="0 0 1" />
       <limit lower="-3.05" upper="3.05" effort="0" velocity="0" />
     </joint>
     <joint name="${arm_id}_joint_6" type="revolute">
-      <origin xyz="0 -0.055 0.0567" rpy="-1.5708 0 0.785" />
+      <origin xyz="0 0.055 0.0567" rpy="${-pi/2} 0 0" />
       <parent link="${arm_id}_link_5" />
       <child link="${arm_id}_link_6" />
-      <axis xyz="0 -1 0" />
+      <axis xyz="0 0 1" />
       <limit lower="-3.05" upper="3.05" effort="0" velocity="0" />
     </joint>
     <joint name="${arm_id}_joint_7" type="fixed">
-      <origin rpy="0 0 0" xyz="0 -0.018 0"/>
+      <origin rpy="0 0 0" xyz="0 0 0.018"/>
       <parent link="${arm_id}_link_6"/>
       <child link="${arm_id}_gripper_connection"/>
+      <axis xyz="0 0 0" />
     </joint>
-    <!--link name="franka_gripper">
-      <collision>
-        <origin xyz="0 0 0" rpy="0 0 0" />
-        <geometry>
-          <cylinder radius="0.03" length="0.01" />
-        </geometry>
-      </collision>
-      <collision>
-        <origin xyz="0.0424 0.0424 -0.02" rpy="0 0 0" />
-        <geometry>
-          <sphere radius="0.03" />
-        </geometry>
-      </collision>
-      <collision>
-        <origin xyz="0.0424 0.0424 -0.03" rpy="0 0 0" />
-        <geometry>
-          <sphere radius="0.03" />
-        </geometry>
-      </collision>
-    </link>
-    <joint name="${arm_id}_joint_7" type="fixed">
-      <origin rpy="-0.985 -1.57 2.55" xyz="0 -0.027 0" />
-      <parent link="${arm_id}_link_6" />
-      <child link="franka_gripper" />
-    </joint-->
  </xacro:macro>
 </robot>
