Commit message: Resolve "Update Avena arm meshes and IK code"

File: core/avena_bringup/urdf/avena_arm.xacro (robot description, xacro)
@@ -1,46 +1,20 @@
 <?xml version="1.0" encoding="utf-8"?>
 <robot xmlns:xacro="http://www.ros.org/wiki/xacro" name="avena">
+  <material name="gray">
+    <color rgba="0.5 0.5 0.5 1.0" />
+  </material>
   <xacro:macro name="avena_arm" params="arm_id:='avena' description_pkg:='avena_bringup'">
     <link name="${arm_id}_link_0">
       <visual>
-        <origin xyz="0 0 0.01" rpy="0 0 0" />
+        <origin xyz="0 0 0" rpy="0 0 0" />
         <geometry>
-          <cylinder radius="0.074744" length="0.02"/>
+          <mesh filename="file://$(find ${description_pkg})/urdf/meshes/avena/link_0.stl" scale="0.001 0.001 0.001" />
         </geometry>
-        <material name="">
-          <color rgba="0.5 0.5 0.5 1" />
-        </material>
-      </visual>
-      <visual>
-        <origin xyz="0 0 0.03375" rpy="0 0 0" />
-        <geometry>
-          <cylinder radius="0.06" length="0.0275"/>
-        </geometry>
-        <material name="">
-          <color rgba="0.5 0.5 0.5 1" />
-        </material>
-      </visual>
-      <visual>
-        <origin xyz="0 0 0.0525" rpy="0 0 0" />
-        <geometry>
-          <cylinder radius="0.04125" length="0.0125"/>
-        </geometry>
+        <material name="gray" />
       </visual>
       <collision>
-        <origin xyz="0 0 0.01" rpy="0 0 0" />
+        <origin xyz="0 0 0" rpy="0 0 0" />
         <geometry>
-          <cylinder radius="0.074744" length="0.02"/>
-        </geometry>
-      </collision>
-      <collision>
-        <origin xyz="0 0 0.03375" rpy="0 0 0" />
-        <geometry>
-          <cylinder radius="0.06" length="0.0275"/>
-        </geometry>
-      </collision>
-      <collision>
-        <origin xyz="0 0 0.0525" rpy="0 0 0" />
-        <geometry>
-          <cylinder radius="0.04125" length="0.0125"/>
+          <mesh filename="file://$(find ${description_pkg})/urdf/meshes/avena/link_0.stl" scale="0.001 0.001 0.001" />
         </geometry>
       </collision>
@@ -48,31 +22,14 @@
     <link name="${arm_id}_link_1">
       <visual>
-        <origin xyz="0 0 -0.06" rpy="0 0 0" />
+        <origin xyz="0 0 0.0495" rpy="${pi} 0 ${-pi/2}" />
         <geometry>
-          <cylinder radius="0.0455" length="0.12" />
+          <mesh filename="file://$(find ${description_pkg})/urdf/meshes/avena/link_1.stl" scale="0.001 0.001 0.001" />
         </geometry>
-        <material name="">
-          <color rgba="0.5 0.5 0.5 1" />
-        </material>
-      </visual>
-      <visual>
-        <origin xyz="0 0.03 -0.0675" rpy="${pi/2} 0 0" />
-        <geometry>
-          <cylinder radius="0.045" length="0.06" />
-        </geometry>
-        <material name="">
-          <color rgba="0.5 0.5 0.5 1" />
-        </material>
+        <material name="gray" />
       </visual>
       <collision>
-        <origin xyz="0 0 -0.06" rpy="0 0 0" />
+        <origin xyz="0 0 0.0495" rpy="${pi} 0 ${-pi/2}" />
         <geometry>
-          <cylinder radius="0.0455" length="0.12" />
-        </geometry>
-      </collision>
-      <collision>
-        <origin xyz="0 0.03 -0.0675" rpy="${pi/2} 0 0" />
-        <geometry>
-          <cylinder radius="0.045" length="0.06" />
+          <mesh filename="file://$(find ${description_pkg})/urdf/meshes/avena/link_1.stl" scale="0.001 0.001 0.001" />
         </geometry>
       </collision>
@@ -80,46 +37,14 @@
     <link name="${arm_id}_link_2">
       <visual>
-        <origin xyz="0 0 0.06" rpy="0 0 0" />
+        <origin xyz="0 0 0.0495" rpy="0 ${pi} ${pi/2}" />
         <geometry>
-          <cylinder radius="0.045" length="0.12" />
+          <mesh filename="file://$(find ${description_pkg})/urdf/meshes/avena/link_2.stl" scale="0.001 0.001 0.001" />
         </geometry>
-        <material name="">
-          <color rgba="0.5 0.5 0.5 1" />
-        </material>
-      </visual>
-      <visual>
-        <origin xyz="0 0.225 0.0675" rpy="${-pi/2} 0 0" />
-        <geometry>
-          <cylinder radius="0.045" length="0.45" />
-        </geometry>
-        <material name="">
-          <color rgba="0.5 0.5 0.5 1" />
-        </material>
-      </visual>
-      <visual>
-        <origin xyz="0 0.4525 0.06" rpy="0 0 0" />
-        <geometry>
-          <cylinder radius="0.045" length="0.12" />
-        </geometry>
-        <material name="">
-          <color rgba="0.5 0.5 0.5 1" />
-        </material>
+        <material name="gray" />
       </visual>
       <collision>
-        <origin xyz="0 0 0.06" rpy="0 0 0" />
+        <origin xyz="0 0 0.0495" rpy="0 ${pi} ${pi/2}" />
         <geometry>
-          <cylinder radius="0.045" length="0.12" />
-        </geometry>
-      </collision>
-      <collision>
-        <origin xyz="0 0.225 0.0675" rpy="${-pi/2} 0 0" />
-        <geometry>
-          <cylinder radius="0.045" length="0.45" />
-        </geometry>
-      </collision>
-      <collision>
-        <origin xyz="0 0.4525 0.06" rpy="0 0 0" />
-        <geometry>
-          <cylinder radius="0.045" length="0.12" />
+          <mesh filename="file://$(find ${description_pkg})/urdf/meshes/avena/link_2.stl" scale="0.001 0.001 0.001" />
         </geometry>
       </collision>
@@ -127,46 +52,14 @@
     <link name="${arm_id}_link_3">
       <visual>
-        <origin xyz="0 0 -0.0475" rpy="0 0 0" />
+        <origin xyz="0 0 0.0721" rpy="0 ${pi} ${-pi/2}" />
         <geometry>
-          <cylinder radius="0.045" length="0.12" />
+          <mesh filename="file://$(find ${description_pkg})/urdf/meshes/avena/link_3.stl" scale="0.001 0.001 0.001" />
         </geometry>
-        <material name="">
-          <color rgba="0.5 0.5 0.5 1" />
-        </material>
-      </visual>
-      <visual>
-        <origin xyz="0 0.225 -0.056" rpy="${-pi/2} 0 0" />
-        <geometry>
-          <cylinder radius="0.045" length="0.45" />
-        </geometry>
-        <material name="">
-          <color rgba="0.5 0.5 0.5 1" />
-        </material>
-      </visual>
-      <visual>
-        <origin xyz="0 0.4475 -0.045" rpy="0 0 0" />
-        <geometry>
-          <cylinder radius="0.04" length="0.115" />
-        </geometry>
-        <material name="">
-          <color rgba="0.5 0.5 0.5 1" />
-        </material>
+        <material name="gray" />
       </visual>
       <collision>
-        <origin xyz="0 0 -0.0475" rpy="0 0 0" />
+        <origin xyz="0 0 0.0721" rpy="0 ${pi} ${-pi/2}" />
         <geometry>
-          <cylinder radius="0.045" length="0.12" />
-        </geometry>
-      </collision>
-      <collision>
-        <origin xyz="0 0.225 -0.056" rpy="${-pi/2} 0 0" />
-        <geometry>
-          <cylinder radius="0.045" length="0.45" />
-        </geometry>
-      </collision>
-      <collision>
-        <origin xyz="0 0.4475 -0.045" rpy="0 0 0" />
-        <geometry>
-          <cylinder radius="0.04" length="0.115" />
+          <mesh filename="file://$(find ${description_pkg})/urdf/meshes/avena/link_3.stl" scale="0.001 0.001 0.001" />
         </geometry>
       </collision>
@@ -174,31 +67,14 @@
     <link name="${arm_id}_link_4">
       <visual>
-        <origin xyz="0 0.0125 0.055" rpy="${pi/2} 0 0" />
+        <origin xyz="0 0 0.064" rpy="${pi/2} 0 ${pi/2}" />
         <geometry>
-          <cylinder radius="0.04" length="0.115" />
+          <mesh filename="file://$(find ${description_pkg})/urdf/meshes/avena/link_4.stl" scale="0.001 0.001 0.001" />
         </geometry>
-        <material name="">
-          <color rgba="0.5 0.5 0.5 1" />
-        </material>
-      </visual>
-      <visual>
-        <origin xyz="0 0 0.025" rpy="0 0 0" />
-        <geometry>
-          <cylinder radius="0.04" length="0.05" />
-        </geometry>
-        <material name="">
-          <color rgba="0.5 0.5 0.5 1" />
-        </material>
+        <material name="gray" />
       </visual>
       <collision>
-        <origin xyz="0 0.0125 0.055" rpy="${pi/2} 0 0" />
+        <origin xyz="0 0 0" rpy="0 0 0" />
         <geometry>
-          <cylinder radius="0.04" length="0.115" />
-        </geometry>
-      </collision>
-      <collision>
-        <origin xyz="0 0 0.025" rpy="0 0 0" />
-        <geometry>
-          <cylinder radius="0.04" length="0.05" />
+          <mesh filename="file://$(find ${description_pkg})/urdf/meshes/avena/link_4.stl" scale="0.001 0.001 0.001" />
         </geometry>
       </collision>
@@ -206,31 +82,14 @@
     <link name="${arm_id}_link_5">
       <visual>
-        <origin xyz="0 0 0.025" rpy="0 0 0" />
+        <origin xyz="0 0 0.064" rpy="${pi/2} 0 ${pi/2}" />
         <geometry>
-          <cylinder radius="0.04" length="0.05" />
+          <mesh filename="file://$(find ${description_pkg})/urdf/meshes/avena/link_5.stl" scale="0.001 0.001 0.001" />
         </geometry>
-        <material name="">
-          <color rgba="0.5 0.5 0.5 1" />
-        </material>
-      </visual>
-      <visual>
-        <origin xyz="0 0.011 0.055" rpy="${pi/2} 0 0" />
-        <geometry>
-          <cylinder radius="0.04" length="0.115" />
-        </geometry>
-        <material name="">
-          <color rgba="0.5 0.5 0.5 1" />
-        </material>
+        <material name="gray" />
       </visual>
       <collision>
-        <origin xyz="0 0 0.025" rpy="0 0 0" />
+        <origin xyz="0 0 0" rpy="0 0 0" />
         <geometry>
-          <cylinder radius="0.04" length="0.05" />
-        </geometry>
-      </collision>
-      <collision>
-        <origin xyz="0 0.011 0.055" rpy="${pi/2} 0 0" />
-        <geometry>
-          <cylinder radius="0.04" length="0.115" />
+          <mesh filename="file://$(find ${description_pkg})/urdf/meshes/avena/link_5.stl" scale="0.001 0.001 0.001" />
         </geometry>
       </collision>
@@ -238,16 +97,14 @@
     <link name="${arm_id}_link_6">
       <visual>
-        <origin xyz="0 0 0.0088" rpy="0 0 0" />
+        <origin xyz="0 0 0" rpy="0 0 0" />
         <geometry>
-          <cylinder radius="0.04" length="0.018" />
+          <mesh filename="file://$(find ${description_pkg})/urdf/meshes/avena/link_6.stl" scale="0.001 0.001 0.001" />
         </geometry>
-        <material name="">
-          <color rgba="0.5 0.5 0.5 1" />
-        </material>
+        <material name="gray" />
       </visual>
       <collision>
-        <origin xyz="0 0 0.0088" rpy="0 0 0" />
+        <origin xyz="0 0 0" rpy="0 0 0" />
         <geometry>
-          <cylinder radius="0.04" length="0.018" />
+          <mesh filename="file://$(find ${description_pkg})/urdf/meshes/avena/link_6.stl" scale="0.001 0.001 0.001" />
         </geometry>
       </collision>
@@ -256,5 +113,5 @@
     <!-- Joints -->
     <joint name="${arm_id}_joint_1" type="revolute">
-      <origin xyz="0 0 0.047" rpy="${pi} 0 ${pi/2}" />
+      <origin xyz="0 0 0.063" rpy="0 0 0" />
       <parent link="${arm_id}_link_0" />
       <child link="${arm_id}_link_1" />
@@ -263,5 +120,5 @@
     </joint>
     <joint name="${arm_id}_joint_2" type="revolute">
-      <origin xyz="0 0.048 -0.0679" rpy="-${pi/2} 0 0" />
+      <origin xyz="0.064 0 0.0495" rpy="0 ${pi/2} 0" />
       <parent link="${arm_id}_link_1" />
       <child link="${arm_id}_link_2" />
@@ -270,5 +127,5 @@
     </joint>
     <joint name="${arm_id}_joint_3" type="revolute">
-      <origin xyz="0 0.452 0" rpy="0 0 0" />
+      <origin xyz="-0.452 0 0" rpy="0 ${pi} 0" />
       <parent link="${arm_id}_link_2" />
       <child link="${arm_id}_link_3" />
@@ -277,5 +134,5 @@
     </joint>
     <joint name="${arm_id}_joint_4" type="revolute">
-      <origin xyz="0 0.447 0.0006" rpy="0 0 0" />
+      <origin xyz="0.452 0 0.0226" rpy="${pi} 0 0" />
       <parent link="${arm_id}_link_3" />
       <child link="${arm_id}_link_4" />
@@ -284,5 +141,5 @@
     </joint>
     <joint name="${arm_id}_joint_5" type="revolute">
-      <origin xyz="0 0.0567 0.055" rpy="${pi/2} 0 ${pi}" />
+      <origin xyz="0.0495 0 0.064" rpy="0 ${pi/2} 0" />
       <parent link="${arm_id}_link_4" />
       <child link="${arm_id}_link_5" />
@@ -291,5 +148,5 @@
     </joint>
     <joint name="${arm_id}_joint_6" type="revolute">
-      <origin xyz="0 0.055 0.0567" rpy="${-pi/2} 0 0" />
+      <origin xyz="0.0495 0 0.064" rpy="0 ${pi/2} 0" />
       <parent link="${arm_id}_link_5" />
       <child link="${arm_id}_link_6" />
@@ -298,5 +155,5 @@
     </joint>
     <joint name="${arm_id}_joint_7" type="fixed">
-      <origin rpy="0 0 0" xyz="0 0 0.018"/>
+      <origin rpy="0 0 0" xyz="0 0 0.0181"/>
       <parent link="${arm_id}_link_6"/>
       <child link="${arm_id}_gripper_connection"/>

File: core/avena_bringup/urdf/avena_arm_ik_fast.urdf (robot description, URDF)
Before this commit: robot avena, 8 links, 7 joints
Joints:
- joint left_avena_joint_1: origin xyz=0 0 0.047 rpy=3.141592653589793 0 1.5707963267948966 -> xyz=0 0 0.063 rpy=0 0 0
- joint left_avena_joint_2: origin xyz=0 0.048 -0.0679 rpy=-1.5707963267948966 0 0 -> xyz=0.064 0 0.0495 rpy=0 1.5707963267948966 0
- joint left_avena_joint_3: origin xyz=0 0.452 0 rpy=0 0 0 -> xyz=-0.452 0 0 rpy=0 3.141592653589793 0
- joint left_avena_joint_4: origin xyz=0 0.447 0.0006 rpy=0 0 0 -> xyz=0.452 0 0.0226 rpy=3.141592653589793 0 0
- joint left_avena_joint_5: origin xyz=0 0.0567 0.055 rpy=1.5707963267948966 0 3.141592653589793 -> xyz=0.0495 0 0.064 rpy=0 1.5707963267948966 0
- joint left_avena_joint_6: origin xyz=0 0.055 0.0567 rpy=-1.5707963267948966 0 0 -> xyz=0.0495 0 0.064 rpy=0 1.5707963267948966 0
- joint left_avena_joint_7: origin xyz=0 0 0.018 rpy=0 0 0 -> xyz=0 0 0.0181 rpy=0 0 0

File: core/avena_bringup/urdf/franka_arm.xacro (robot description, xacro)
@@ -8,10 +8,10 @@
       <visual>
         <geometry>
-          <mesh filename="file://$(find ${description_pkg})/urdf/meshes/visual/link0.dae"/>
+          <mesh filename="file://$(find ${description_pkg})/urdf/meshes/franka/link0.dae"/>
         </geometry>
       </visual>
       <collision>
         <geometry>
-          <mesh filename="file://$(find ${description_pkg})/urdf/meshes/visual/link0.dae"/>
+          <mesh filename="file://$(find ${description_pkg})/urdf/meshes/franka/link0.dae"/>
         </geometry>
       </collision>
@@ -20,10 +20,10 @@
       <visual>
         <geometry>
-          <mesh filename="file://$(find ${description_pkg})/urdf/meshes/visual/link1.dae"/>
+          <mesh filename="file://$(find ${description_pkg})/urdf/meshes/franka/link1.dae"/>
         </geometry>
       </visual>
       <collision>
         <geometry>
-          <mesh filename="file://$(find ${description_pkg})/urdf/meshes/visual/link1.dae"/>
+          <mesh filename="file://$(find ${description_pkg})/urdf/meshes/franka/link1.dae"/>
         </geometry>
       </collision>
@@ -32,10 +32,10 @@
       <visual>
         <geometry>
-          <mesh filename="file://$(find ${description_pkg})/urdf/meshes/visual/link2.dae"/>
+          <mesh filename="file://$(find ${description_pkg})/urdf/meshes/franka/link2.dae"/>
         </geometry>
       </visual>
       <collision>
         <geometry>
-          <mesh filename="file://$(find ${description_pkg})/urdf/meshes/visual/link2.dae"/>
+          <mesh filename="file://$(find ${description_pkg})/urdf/meshes/franka/link2.dae"/>
         </geometry>
       </collision>
@@ -44,10 +44,10 @@
       <visual>
         <geometry>
-          <mesh filename="file://$(find ${description_pkg})/urdf/meshes/visual/link3.dae"/>
+          <mesh filename="file://$(find ${description_pkg})/urdf/meshes/franka/link3.dae"/>
         </geometry>
       </visual>
       <collision>
         <geometry>
-          <mesh filename="file://$(find ${description_pkg})/urdf/meshes/visual/link3.dae"/>
+          <mesh filename="file://$(find ${description_pkg})/urdf/meshes/franka/link3.dae"/>
         </geometry>
       </collision>
@@ -56,10 +56,10 @@
       <visual>
         <geometry>
-          <mesh filename="file://$(find ${description_pkg})/urdf/meshes/visual/link4.dae"/>
+          <mesh filename="file://$(find ${description_pkg})/urdf/meshes/franka/link4.dae"/>
         </geometry>
       </visual>
       <collision>
         <geometry>
-          <mesh filename="file://$(find ${description_pkg})/urdf/meshes/visual/link4.dae"/>
+          <mesh filename="file://$(find ${description_pkg})/urdf/meshes/franka/link4.dae"/>
         </geometry>
       </collision>
@@ -68,10 +68,10 @@
       <visual>
         <geometry>
-          <mesh filename="file://$(find ${description_pkg})/urdf/meshes/visual/link5.dae"/>
+          <mesh filename="file://$(find ${description_pkg})/urdf/meshes/franka/link5.dae"/>
         </geometry>
       </visual>
       <collision>
         <geometry>
-          <mesh filename="file://$(find ${description_pkg})/urdf/meshes/visual/link5.dae"/>
+          <mesh filename="file://$(find ${description_pkg})/urdf/meshes/franka/link5.dae"/>
         </geometry>
       </collision>
@@ -80,10 +80,10 @@
       <visual>
         <geometry>
-          <mesh filename="file://$(find ${description_pkg})/urdf/meshes/visual/link6.dae"/>
+          <mesh filename="file://$(find ${description_pkg})/urdf/meshes/franka/link6.dae"/>
         </geometry>
       </visual>
       <collision>
         <geometry>
-          <mesh filename="file://$(find ${description_pkg})/urdf/meshes/visual/link6.dae"/>
+          <mesh filename="file://$(find ${description_pkg})/urdf/meshes/franka/link6.dae"/>
         </geometry>
       </collision>
@@ -92,10 +92,10 @@
       <visual>
         <geometry>
-          <mesh filename="file://$(find ${description_pkg})/urdf/meshes/visual/link7.dae"/>
+          <mesh filename="file://$(find ${description_pkg})/urdf/meshes/franka/link7.dae"/>
         </geometry>
       </visual>
       <collision>
         <geometry>
-          <mesh filename="file://$(find ${description_pkg})/urdf/meshes/visual/link7.dae"/>
+          <mesh filename="file://$(find ${description_pkg})/urdf/meshes/franka/link7.dae"/>
         </geometry>
       </collision>

Commit message: Merge arm_controller into develop

File: core/avena_bringup/urdf/avena_arm.xacro (robot description, xacro)
@@ -13,4 +13,9 @@
         <material name="gray" />
       </visual>
+      <inertial>
+        <origin xyz="0. -0.0129 0.00034" rpy="0. 0. 0."/>
+        <mass value="0.75"/>
+        <inertia ixx="1."  ixy="0."  ixz="0." iyy="1." iyz="0." izz="1." />
+      </inertial>
       <collision>
         <origin xyz="0 0 0" rpy="0 0 0" />
@@ -28,4 +33,9 @@
         <material name="gray" />
       </visual>
+      <inertial>
+        <origin xyz="0.019 0. 0.0445 " rpy="0. 0. ${pi/2}"/>
+        <mass value="1.798"/>
+        <inertia ixx="2.233e-03"  ixy="0."  ixz="0." iyy="2.047e-03" iyz="0." izz="2.384e-03" />
+      </inertial>
       <collision>
         <origin xyz="0 0 0.0495" rpy="${pi} 0 ${-pi/2}" />
@@ -43,4 +53,9 @@
         <material name="gray" />
       </visual>
+      <inertial>
+        <origin xyz="-0.226 0 0.0334" rpy="0. 0. ${pi/2}"/>
+        <mass value="4.406"/>
+        <inertia ixx="1.941e-01"  ixy="0."  ixz="0." iyy="5.522e-03" iyz="0." izz="1.941e-01" />
+      </inertial>
       <collision>
         <origin xyz="0 0 0.0495" rpy="0 ${pi} ${pi/2}" />
@@ -52,5 +67,5 @@
     <link name="${arm_id}_link_3">
       <visual>
-        <origin xyz="0 0 0.0721" rpy="0 ${pi} ${-pi/2}" />
+        <origin xyz="0. 0. 0.0721" rpy="0 ${pi} ${-pi/2}" />
         <geometry>
           <mesh filename="file://$(find ${description_pkg})/urdf/meshes/avena/link_3.stl" scale="0.001 0.001 0.001" />
@@ -58,4 +73,9 @@
         <material name="gray" />
       </visual>
+      <inertial>
+        <origin xyz="0.3046 0. 0.0588" rpy="0 0 ${pi/2}"/>
+        <mass value="3.267"/>
+        <inertia ixx="1.149e-01"  ixy="0"  ixz="0" iyy="4.518e-03" iyz="0" izz="1.148e-01" />
+      </inertial>
       <collision>
         <origin xyz="0 0 0.0721" rpy="0 ${pi} ${-pi/2}" />
@@ -73,4 +93,9 @@
         <material name="gray" />
       </visual>
+      <inertial>
+        <origin xyz="0.019 0. 0.059 " rpy="0. 0. ${pi/2}"/>
+        <mass value="1.798"/>
+        <inertia ixx="2.233e-03"  ixy="0."  ixz="0." iyy="2.047e-03" iyz="0." izz="2.384e-03" />
+      </inertial>
       <collision>
         <origin xyz="0 0 0" rpy="0 0 0" />
@@ -88,4 +113,9 @@
         <material name="gray" />
       </visual>
+      <inertial>
+        <origin xyz="0.019 0 0.059" rpy="0. 0. ${pi/2}"/>
+        <mass value="1.798"/>
+        <inertia ixx="2.233e-03"  ixy="0."  ixz="0." iyy="2.047e-03" iyz="0." izz="2.384e-03" />
+      </inertial>
       <collision>
         <origin xyz="0 0 0" rpy="0 0 0" />
@@ -103,4 +133,9 @@
         <material name="gray" />
       </visual>
+      <inertial>
+        <origin xyz="0 0 0" rpy="0 0 0"/>
+        <mass value="8.200e-02"/>
+        <inertia ixx="4.100e-05"  ixy="0"  ixz="0" iyy="4.200e-05" iyz="0" izz="8.000e-05" />
+      </inertial>
       <collision>
         <origin xyz="0 0 0" rpy="0 0 0" />
@@ -117,5 +152,5 @@
       <child link="${arm_id}_link_1" />
       <axis xyz="0 0 1" />
-      <limit lower="-3.05" upper="3.05" effort="0" velocity="0" />
+      <limit lower="-3.05" upper="3.05" effort="80" velocity="0" />
     </joint>
     <joint name="${arm_id}_joint_2" type="revolute">
@@ -124,5 +159,5 @@
       <child link="${arm_id}_link_2" />
       <axis xyz="0 0 1" />
-      <limit lower="-1.57" upper="1.57" effort="0" velocity="0" />
+      <limit lower="-1.57" upper="1.57" effort="120" velocity="0" />
     </joint>
     <joint name="${arm_id}_joint_3" type="revolute">
@@ -131,5 +166,5 @@
       <child link="${arm_id}_link_3" />
       <axis xyz="0 0 1" />
-      <limit lower="-2.9" upper="2.9" effort="0" velocity="0" />
+      <limit lower="-2.9" upper="2.9" effort="80" velocity="0" />
     </joint>
     <joint name="${arm_id}_joint_4" type="revolute">
@@ -138,5 +173,5 @@
       <child link="${arm_id}_link_4" />
       <axis xyz="0 0 1" />
-      <limit lower="-3.05" upper="3.05" effort="0" velocity="0" />
+      <limit lower="-3.05" upper="3.05" effort="60" velocity="0" />
     </joint>
     <joint name="${arm_id}_joint_5" type="revolute">
@@ -145,5 +180,5 @@
       <child link="${arm_id}_link_5" />
       <axis xyz="0 0 1" />
-      <limit lower="-3.05" upper="3.05" effort="0" velocity="0" />
+      <limit lower="-3.05" upper="3.05" effort="40" velocity="0" />
     </joint>
     <joint name="${arm_id}_joint_6" type="revolute">
@@ -152,5 +187,5 @@
       <child link="${arm_id}_link_6" />
       <axis xyz="0 0 1" />
-      <limit lower="-3.05" upper="3.05" effort="0" velocity="0" />
+      <limit lower="-3.05" upper="3.05" effort="40" velocity="0" />
     </joint>
     <joint name="${arm_id}_joint_7" type="fixed">
