Commit message: Loading world from urdf instead of using bullet api to create world; change...

File: core/avena_bringup/urdf/avena_arm.xacro (robot description, xacro)
@@ -5,4 +5,6 @@
   </material>
   <xacro:macro name="avena_arm" params="arm_id:='avena' description_pkg:='avena_bringup'">
+    <!-- Links -->
+    <link name="base_link" />
     <link name="${arm_id}_link_0">
       <visual>
@@ -99,5 +101,5 @@
       </inertial>
       <collision>
-        <origin xyz="0 0 0" rpy="0 0 0" />
+        <origin xyz="0 0 0.064" rpy="${pi/2} 0 ${pi/2}" />
         <geometry>
           <mesh filename="file://$(find ${description_pkg})/urdf/meshes/avena/link_4.stl" scale="0.001 0.001 0.001" />
@@ -119,5 +121,5 @@
       </inertial>
       <collision>
-        <origin xyz="0 0 0" rpy="0 0 0" />
+        <origin xyz="0 0 0.064" rpy="${pi/2} 0 ${pi/2}" />
         <geometry>
           <mesh filename="file://$(find ${description_pkg})/urdf/meshes/avena/link_5.stl" scale="0.001 0.001 0.001" />
@@ -147,4 +149,10 @@
     <link name="${arm_id}_gripper_connection"/>
     <!-- Joints -->
+    <joint name="base_joint" type="fixed">
+      <origin rpy="0 0 0" xyz="0 0 0"/>
+      <parent link="base_link"/>
+      <child link="${arm_id}_link_0"/>
+      <axis xyz="0 0 0"/>
+    </joint>
     <joint name="${arm_id}_joint_1" type="revolute">
       <origin xyz="0 0 0.063" rpy="0 0 0" />

File: core/avena_bringup/urdf/franka_arm.xacro (robot description, xacro)
@@ -4,6 +4,7 @@
   <!-- arm_id: Namespace of the franka arm. Serves to differentiate between arms in case of multiple instances. -->
   <xacro:macro name="franka_arm" params="arm_id:='franka' description_pkg:='avena_bringup' connected_to:='' xyz:='0 0 0' rpy:='0 0 0' safety_distance:=0">
-  <!-- Links   -->
-  <link name="${arm_id}_link_0">
+    <!-- Links -->
+    <link name="base_link" />
+    <link name="${arm_id}_link_0">
       <visual>
         <geometry>
@@ -103,11 +104,10 @@
     <link name="${arm_id}_gripper_connection"/>
     <!-- Joints -->
-    <xacro:unless value="${not connected_to}">
-      <joint name="${arm_id}_joint__${connected_to}" type="fixed">
-        <parent link="${connected_to}"/>
-        <child link="${arm_id}_link_0"/>
-        <origin rpy="${rpy}" xyz="${xyz}"/>
-      </joint>
-    </xacro:unless>
+    <joint name="base_joint" type="fixed">
+      <origin rpy="0 0 0" xyz="0 0 0"/>
+      <parent link="base_link"/>
+      <child link="${arm_id}_link_0"/>
+      <axis xyz="0 0 0"/>
+    </joint>
     <joint name="${arm_id}_joint_1" type="revolute">
       <safety_controller k_position="100.0" k_velocity="40.0" soft_lower_limit="-2.8973" soft_upper_limit="2.8973"/>

Commit message: Merge branch 'arm_controller' into 'develop'

File: core/avena_bringup/urdf/avena_arm.xacro (robot description, xacro)
@@ -37,5 +37,5 @@
       <inertial>
         <origin xyz="0.019 0. 0.0445 " rpy="0. 0. ${pi/2}"/>
-        <mass value="1.798"/>
+        <mass value="1.9"/>
         <inertia ixx="2.233e-03"  ixy="0."  ixz="0." iyy="2.047e-03" iyz="0." izz="2.384e-03" />
       </inertial>
@@ -57,5 +57,5 @@
       <inertial>
         <origin xyz="-0.226 0 0.0334" rpy="0. 0. ${pi/2}"/>
-        <mass value="4.406"/>
+        <mass value="4.6"/>
         <inertia ixx="1.941e-01"  ixy="0."  ixz="0." iyy="5.522e-03" iyz="0." izz="1.941e-01" />
       </inertial>
@@ -77,5 +77,5 @@
       <inertial>
         <origin xyz="0.3046 0. 0.0588" rpy="0 0 ${pi/2}"/>
-        <mass value="3.267"/>
+        <mass value="3.4"/>
         <inertia ixx="1.149e-01"  ixy="0"  ixz="0" iyy="4.518e-03" iyz="0" izz="1.148e-01" />
       </inertial>
@@ -97,5 +97,5 @@
       <inertial>
         <origin xyz="0.019 0. 0.059 " rpy="0. 0. ${pi/2}"/>
-        <mass value="1.798"/>
+        <mass value="1.9"/>
         <inertia ixx="2.233e-03"  ixy="0."  ixz="0." iyy="2.047e-03" iyz="0." izz="2.384e-03" />
       </inertial>
@@ -117,5 +117,5 @@
       <inertial>
         <origin xyz="0.019 0 0.059" rpy="0. 0. ${pi/2}"/>
-        <mass value="1.798"/>
+        <mass value="1.9"/>
         <inertia ixx="2.233e-03"  ixy="0."  ixz="0." iyy="2.047e-03" iyz="0." izz="2.384e-03" />
       </inertial>
@@ -167,5 +167,5 @@
       <child link="${arm_id}_link_2" />
       <axis xyz="0 0 1" />
-      <limit lower="-1.57" upper="1.57" effort="120" velocity="0" />
+      <limit lower="-1.57" upper="1.57" effort="160" velocity="0" />
     </joint>
     <joint name="${arm_id}_joint_3" type="revolute">

Commit message: cartesian_error

File: core/avena_bringup/urdf/avena_arm.xacro (robot description, xacro)
@@ -156,5 +156,5 @@
     </joint>
     <joint name="${arm_id}_joint_1" type="revolute">
-      <origin xyz="0 0 0.063" rpy="0 0 0" />
+      <origin xyz="0 0 0.063" rpy="0 0 -0.1963" />
       <parent link="${arm_id}_link_0" />
       <child link="${arm_id}_link_1" />

Commit message: Bs change scene

File: core/avena_bringup/urdf/avena_arm.xacro (robot description, xacro)
@@ -6,5 +6,5 @@
   <xacro:macro name="avena_arm" params="arm_id:='avena' description_pkg:='avena_bringup'">
     <!-- Links -->
-    <link name="base_link" />
+    <link name="robot_base_link" />
     <link name="${arm_id}_link_0">
       <visual>
@@ -151,10 +151,10 @@
     <joint name="base_joint" type="fixed">
       <origin rpy="0 0 0" xyz="0 0 0"/>
-      <parent link="base_link"/>
+      <parent link="robot_base_link"/>
       <child link="${arm_id}_link_0"/>
       <axis xyz="0 0 0"/>
     </joint>
     <joint name="${arm_id}_joint_1" type="revolute">
-      <origin xyz="0 0 0.063" rpy="0 0 0" />
+      <origin xyz="0 0 0.063" rpy="0 0 -0.1963" /> <!-- Offset from position -->
       <parent link="${arm_id}_link_0" />
       <child link="${arm_id}_link_1" />

File: core/avena_bringup/urdf/franka_arm.xacro (robot description, xacro)
@@ -5,5 +5,5 @@
   <xacro:macro name="franka_arm" params="arm_id:='franka' description_pkg:='avena_bringup' connected_to:='' xyz:='0 0 0' rpy:='0 0 0' safety_distance:=0">
     <!-- Links -->
-    <link name="base_link" />
+    <link name="robot_base_link" />
     <link name="${arm_id}_link_0">
       <visual>
@@ -106,5 +106,5 @@
     <joint name="base_joint" type="fixed">
       <origin rpy="0 0 0" xyz="0 0 0"/>
-      <parent link="base_link"/>
+      <parent link="robot_base_link"/>
       <child link="${arm_id}_link_0"/>
       <axis xyz="0 0 0"/>

File: core/avena_bringup/urdf/franka_calibration.urdf.xacro (robot description, xacro)
@@ -10,5 +10,5 @@
   <xacro:property name="x_axis_offset" value="${grid_size}" />
   <xacro:property name="y_axis_offset" value="${1.5 * grid_size}" />
-  <xacro:property name="z_axis_offset" value="0.02306" />
+  <xacro:property name="z_axis_offset" value="0.02506" />
   <xacro:property name="x_axis_rot" value="${pi}" />
   <xacro:property name="y_axis_rot" value="0" />

File: core/avena_bringup/worlds/avena_table.xacro (robot description, xacro)
@@ -1,10 +1,6 @@
 <?xml version="1.0" encoding="utf-8"?>
 <robot xmlns:xacro="http://www.ros.org/wiki/xacro" name="table">
-  <!-- Constants -->
-  <material name="transparent">
-    <color rgba="1 1 1 0.2" />
-  </material>
   <!-- Collision box -->
-  <xacro:macro name="collision_box" params="name size visual:='true' transparent:='false' xyz:='0 0 0' rpy:='0 0 0' rgba:='0.8 0.8 0.8 1' table_base_link:='table_base_link'">
+  <xacro:macro name="collision_box" params="name size visual:='true' xyz:='0 0 0' rpy:='0 0 0' rgba:='0.8 0.8 0.8 1' table_base_link:='table_base_link'">
     <joint name="${name}" type="fixed">
       <origin xyz="${xyz}" rpy="${rpy}" />
@@ -18,12 +14,7 @@
             <box size="${size}"/>
           </geometry>
-          <xacro:if value="${transparent}">
-            <material name="transparent" />
-          </xacro:if>
-          <xacro:unless value="${transparent}">
-            <material name="custom_color">
-              <color rgba="${rgba}" />
-            </material>
-          </xacro:unless>
+          <material name="">
+            <color rgba="${rgba}" />
+          </material>
         </visual>
       </xacro:if>
@@ -35,14 +26,14 @@
     </link>
   </xacro:macro>
-  <!-- Table -->
+ <!-- Table -->
   <xacro:macro name="table" params="x_min:=0 x_max:=0 y_min:=0 y_max:=0">
-    <xacro:property name="thickness" value="0.01" />
-    <xacro:property name="walls_height" value="1.5" />
+    <xacro:property name="wall_thickness" value="0.01" />
+    <xacro:property name="walls_height" value="1.7" />
     <xacro:property name="x_origin" value="${(x_max + x_min) / 2}" />
     <xacro:property name="y_origin" value="${(y_max + y_min) / 2}" />
     <xacro:property name="x_dim" value="${x_max - x_min}" />
     <xacro:property name="y_dim" value="${y_max - y_min}" />
-    <xacro:property name="camera_stick_size" value="0.05" />
-    <xacro:property name="camera_stick_height" value="${walls_height}" />
+    <xacro:property name="stick_size" value="0.05" />
+    <xacro:property name="stick_height" value="${walls_height}" />
     <xacro:property name="camera_size" value="0.1" />
     <xacro:property name="camera_height" value="1.05" />
@@ -51,6 +42,6 @@
     <xacro:collision_box
       name="table_top"
-      xyz="${x_origin} ${y_origin} ${-thickness / 2}"
-      size="${x_dim} ${y_dim} ${thickness}"
+      xyz="${x_origin} ${y_origin} ${-wall_thickness / 2}"
+      size="${x_dim} ${y_dim} ${wall_thickness}"
       rgba="1 0.6 0.5 1"
     />
@@ -59,65 +50,88 @@
     <xacro:collision_box
       name="front_wall"
-      xyz="${1 + thickness / 2} ${y_origin} ${walls_height / 2}"
-      size="${thickness} ${y_dim} ${walls_height}"
-      transparent="true"
+      xyz="${x_dim + wall_thickness / 2} ${y_origin} ${walls_height / 2}"
+      size="${wall_thickness} ${y_dim} ${walls_height}"
       visual="false"
     />
     <xacro:collision_box
       name="back_wall"
-      xyz="${-thickness / 2} ${y_origin} ${walls_height / 2}"
-      size="${thickness} ${y_dim} ${walls_height}"
-      transparent="true"
+      xyz="${-wall_thickness / 2} ${y_origin} ${walls_height / 2}"
+      size="${wall_thickness} ${y_dim} ${walls_height}"
+      visual="false"
     />
     <xacro:collision_box
       name="left_side_wall"
-      xyz="${x_dim / 2} ${y_max + thickness / 2} ${walls_height / 2}"
-      size="${x_dim} ${thickness} ${walls_height}"
-      transparent="true"
+      xyz="${x_dim / 2} ${y_max + wall_thickness / 2} ${walls_height / 2}"
+      size="${x_dim} ${wall_thickness} ${walls_height}"
+      visual="false"
     />
     <xacro:collision_box
       name="right_side_wall"
-      xyz="${x_dim / 2} ${y_min - thickness / 2} ${walls_height / 2}"
-      size="${x_dim} ${thickness} ${walls_height}"
-      transparent="true"
-    />
-    <!-- <xacro:collision_box
-      name="top_wall"
-      xyz="${x_origin} ${y_origin} ${walls_height + thickness / 2}"
-      size="${x_dim} ${y_dim} ${thickness}"
-      transparent="true"
-    /> -->
-    <!-- ******************************************************* -->
-    <!-- <xacro:collision_box
-      name="temporary_wall"
-      xyz="${x_origin + 0.1} ${-0.1} ${walls_height / 2}"
-      size="${x_dim + 0.2} ${thickness} ${walls_height}"
-      transparent="true"
-    /> -->
-    <!-- ******************************************************* -->
-    <!-- ********************************************* -->
-    <!-- CAMERAS STICKS -->
-    <xacro:collision_box
-      name="left_camera_stick"
-      xyz="${x_max - camera_stick_size / 2} ${y_max - camera_stick_size / 2} ${camera_stick_height / 2}"
-      size="${camera_stick_size} ${camera_stick_size} ${camera_stick_height}"
+      xyz="${x_dim / 2} ${y_min - wall_thickness / 2} ${walls_height / 2}"
+      size="${x_dim} ${wall_thickness} ${walls_height}"
+      visual="false"
     />
     <xacro:collision_box
-      name="right_camera_stick"
-      xyz="${x_max - camera_stick_size / 2} ${y_min + camera_stick_size / 2} ${camera_stick_height / 2}"
-      size="${camera_stick_size} ${camera_stick_size} ${camera_stick_height}"
+      name="temp_left_collision_wall_0"
+      xyz="${x_dim / 2} 0.7 ${walls_height / 2}"
+      size="${x_dim} ${wall_thickness} ${walls_height}"
+      rgba="1 1 1 0.2"
+    />
+    <xacro:collision_box
+      name="temp_left_collision_wall_1"
+      xyz="${x_dim / 2} 0.1 ${walls_height / 2}"
+      size="${x_dim} ${wall_thickness} ${walls_height}"
+      rgba="1 1 1 0.2"
+    />
+    <!-- ********************************************* -->
+    <!-- STICKS -->
+    <xacro:collision_box
+      name="left_back"
+      xyz="${stick_size / 2} 0.8 ${stick_height / 2}"
+      size="${stick_size} ${2 * stick_size} ${stick_height}"
+      visual="false"
+    />
+    <xacro:collision_box
+      name="left_front"
+      xyz="${x_dim - stick_size / 2} 0.8 ${stick_height / 2}"
+      size="${stick_size} ${2 * stick_size} ${stick_height}"
+      visual="false"
+    />
+    <xacro:collision_box
+      name="middle_front"
+      xyz="${x_dim - stick_size / 2} 0 ${stick_height / 2}"
+      size="${stick_size} ${2 * stick_size} ${stick_height}"
+      visual="false"
+    />
+    <xacro:collision_box
+      name="middle_back"
+      xyz="${stick_size / 2} 0 ${stick_height / 2}"
+      size="${stick_size} ${2 * stick_size} ${stick_height}"
+      visual="false"
+    />
+    <xacro:collision_box
+      name="right_front"
+      xyz="${x_dim - stick_size / 2} -0.8 ${stick_height / 2}"
+      size="${stick_size} ${2 * stick_size} ${stick_height}"
+      visual="false"
+    />
+    <xacro:collision_box
+      name="right_back"
+      xyz="${stick_size / 2} -0.8 ${stick_height / 2}"
+      size="${stick_size} ${2 * stick_size} ${stick_height}"
+      visual="false"
     />
     <!-- ********************************************* -->
     <!-- CAMERAS -->
-    <xacro:collision_box
+    <!-- <xacro:collision_box
       name="left_camera"
       xyz="${x_max - camera_size / 2} ${y_max - camera_size / 2} ${camera_height}"
       size="${camera_size} ${camera_size} ${camera_size}"
-    />
-    <xacro:collision_box
+    /> -->
+    <!-- <xacro:collision_box
       name="right_camera"
       xyz="${x_max - camera_size / 2} ${y_min + camera_size / 2} ${camera_height}"
       size="${camera_size} ${camera_size} ${camera_size}"
-    />
+    /> -->
   </xacro:macro>
 </robot>

Commit message: params update

File: core/avena_bringup/urdf/avena_arm.xacro (robot description, xacro)
@@ -37,5 +37,5 @@
       <inertial>
         <origin xyz="0.019 0. 0.0445 " rpy="0. 0. ${pi/2}"/>
-        <mass value="1.9"/>
+        <mass value="1.960"/>
         <inertia ixx="2.233e-03"  ixy="0."  ixz="0." iyy="2.047e-03" iyz="0." izz="2.384e-03" />
       </inertial>
@@ -57,5 +57,5 @@
       <inertial>
         <origin xyz="-0.226 0 0.0334" rpy="0. 0. ${pi/2}"/>
-        <mass value="4.6"/>
+        <mass value="4.660"/>
         <inertia ixx="1.941e-01"  ixy="0."  ixz="0." iyy="5.522e-03" iyz="0." izz="1.941e-01" />
       </inertial>
@@ -77,5 +77,5 @@
       <inertial>
         <origin xyz="0.3046 0. 0.0588" rpy="0 0 ${pi/2}"/>
-        <mass value="3.4"/>
+        <mass value="3.375"/>
         <inertia ixx="1.149e-01"  ixy="0"  ixz="0" iyy="4.518e-03" iyz="0" izz="1.148e-01" />
       </inertial>
@@ -97,5 +97,5 @@
       <inertial>
         <origin xyz="0.019 0. 0.059 " rpy="0. 0. ${pi/2}"/>
-        <mass value="1.9"/>
+        <mass value="1.960"/>
         <inertia ixx="2.233e-03"  ixy="0."  ixz="0." iyy="2.047e-03" iyz="0." izz="2.384e-03" />
       </inertial>
@@ -117,5 +117,5 @@
       <inertial>
         <origin xyz="0.019 0 0.059" rpy="0. 0. ${pi/2}"/>
-        <mass value="1.9"/>
+        <mass value="1.960"/>
         <inertia ixx="2.233e-03"  ixy="0."  ixz="0." iyy="2.047e-03" iyz="0." izz="2.384e-03" />
       </inertial>
@@ -184,5 +184,5 @@
     </joint>
     <joint name="${arm_id}_joint_5" type="revolute">
-      <origin xyz="0.0495 0 0.064" rpy="0 ${pi/2} 0" />
+      <origin xyz="0.0495 0 0.064" rpy="0 ${-pi/2} ${pi}" />
       <parent link="${arm_id}_link_4" />
       <child link="${arm_id}_link_5" />

Commit message: ikfast update

File: core/avena_bringup/urdf/avena_arm.xacro (robot description, xacro)
@@ -198,5 +198,5 @@
     </joint>
     <joint name="${arm_id}_joint_7" type="fixed">
-      <origin rpy="0 0 0" xyz="0 0 0.0181"/>
+      <origin xyz="0 0 0.0181" rpy="0 0 0"/>
       <parent link="${arm_id}_link_6"/>
       <child link="${arm_id}_gripper_connection"/>

Commit message: update IKFast generated code

File: core/avena_bringup/urdf/avena_arm.xacro (robot description, xacro)
@@ -37,5 +37,5 @@
       <inertial>
         <origin xyz="0.019 0. 0.0445 " rpy="0. 0. ${pi/2}"/>
-        <mass value="1.9"/>
+        <mass value="1.960"/>
         <inertia ixx="2.233e-03"  ixy="0."  ixz="0." iyy="2.047e-03" iyz="0." izz="2.384e-03" />
       </inertial>
@@ -57,5 +57,5 @@
       <inertial>
         <origin xyz="-0.226 0 0.0334" rpy="0. 0. ${pi/2}"/>
-        <mass value="4.6"/>
+        <mass value="4.660"/>
         <inertia ixx="1.941e-01"  ixy="0."  ixz="0." iyy="5.522e-03" iyz="0." izz="1.941e-01" />
       </inertial>
@@ -77,5 +77,5 @@
       <inertial>
         <origin xyz="0.3046 0. 0.0588" rpy="0 0 ${pi/2}"/>
-        <mass value="3.4"/>
+        <mass value="3.375"/>
         <inertia ixx="1.149e-01"  ixy="0"  ixz="0" iyy="4.518e-03" iyz="0" izz="1.148e-01" />
       </inertial>
@@ -97,5 +97,5 @@
       <inertial>
         <origin xyz="0.019 0. 0.059 " rpy="0. 0. ${pi/2}"/>
-        <mass value="1.9"/>
+        <mass value="1.960"/>
         <inertia ixx="2.233e-03"  ixy="0."  ixz="0." iyy="2.047e-03" iyz="0." izz="2.384e-03" />
       </inertial>
@@ -117,5 +117,5 @@
       <inertial>
         <origin xyz="0.019 0 0.059" rpy="0. 0. ${pi/2}"/>
-        <mass value="1.9"/>
+        <mass value="1.960"/>
         <inertia ixx="2.233e-03"  ixy="0."  ixz="0." iyy="2.047e-03" iyz="0." izz="2.384e-03" />
       </inertial>
@@ -184,5 +184,5 @@
     </joint>
     <joint name="${arm_id}_joint_5" type="revolute">
-      <origin xyz="0.0495 0 0.064" rpy="0 ${pi/2} 0" />
+      <origin xyz="0.0495 0 0.064" rpy="0 ${-pi/2} ${pi}" />
       <parent link="${arm_id}_link_4" />
       <child link="${arm_id}_link_5" />
@@ -198,5 +198,5 @@
     </joint>
     <joint name="${arm_id}_joint_7" type="fixed">
-      <origin rpy="0 0 0" xyz="0 0 0.0181"/>
+      <origin xyz="0 0 0.0181" rpy="0 0 0"/>
       <parent link="${arm_id}_link_6"/>
       <child link="${arm_id}_gripper_connection"/>

Commit message: orientation constraints

File: core/avena_bringup/urdf/avena_arm.xacro (robot description, xacro)
@@ -167,5 +167,5 @@
       <child link="${arm_id}_link_2" />
       <axis xyz="0 0 1" />
-      <limit lower="-1.57" upper="1.57" effort="160" velocity="0" />
+      <limit lower="-1.57" upper="1.57" effort="180" velocity="0" />
     </joint>
     <joint name="${arm_id}_joint_3" type="revolute">
@@ -174,5 +174,5 @@
       <child link="${arm_id}_link_3" />
       <axis xyz="0 0 1" />
-      <limit lower="-2.9" upper="2.9" effort="80" velocity="0" />
+      <limit lower="-2.9" upper="2.9" effort="120" velocity="0" />
     </joint>
     <joint name="${arm_id}_joint_4" type="revolute">

Commit message: partial urdf changes

File: core/avena_bringup/urdf/avena_arm.xacro (robot description, xacro)
@@ -36,7 +36,7 @@
       </visual>
       <inertial>
-        <origin xyz="0.019 0. 0.0445 " rpy="0. 0. ${pi/2}"/>
-        <mass value="1.960"/>
-        <inertia ixx="2.233e-03"  ixy="0."  ixz="0." iyy="2.047e-03" iyz="0." izz="2.384e-03" />
+        <origin xyz="-0.00005 -0.007 0.0175 " rpy="0. 0. ${pi/2}"/>
+        <mass value="3.5"/>
+        <inertia ixx="5.372e-03"  ixy="0."  ixz="0." iyy="4.691e-03" iyz="0." izz="5.059e-03" />
       </inertial>
       <collision>
@@ -56,7 +56,7 @@
       </visual>
       <inertial>
-        <origin xyz="-0.226 0 0.0334" rpy="0. 0. ${pi/2}"/>
-        <mass value="4.660"/>
-        <inertia ixx="1.941e-01"  ixy="0."  ixz="0." iyy="5.522e-03" iyz="0." izz="1.941e-01" />
+        <origin xyz="0. 0.17651 0.015.28" rpy="0. 0. ${pi/2}"/>
+        <mass value="6.3"/>
+        <inertia ixx="2.809e-01"  ixy="0."  ixz="0." iyy="8.463e-03" iyz="0." izz="2.804e-01" />
       </inertial>
       <collision>

Commit message: urdf fix

File: core/avena_bringup/urdf/avena_arm.xacro (robot description, xacro)
@@ -56,5 +56,5 @@
       </visual>
       <inertial>
-        <origin xyz="0. 0.17651 0.015.28" rpy="0. 0. ${pi/2}"/>
+        <origin xyz="0. 0.17651 0.01528" rpy="0. 0. ${pi/2}"/>
         <mass value="6.3"/>
         <inertia ixx="2.809e-01"  ixy="0."  ixz="0." iyy="8.463e-03" iyz="0." izz="2.804e-01" />
