Commit message: update urdf

File: core/avena_bringup/urdf/avena_arm.xacro (robot description, xacro)
@@ -29,5 +29,5 @@
     <link name="${arm_id}_link_1">
       <visual>
-        <origin xyz="0 0 0.0495" rpy="${pi} 0 ${-pi/2}" />
+        <origin xyz="0 0 0.0763" rpy="${pi} 0 ${-pi/2}" />
         <geometry>
           <mesh filename="file://$(find ${description_pkg})/urdf/meshes/avena/link_1.stl" scale="0.001 0.001 0.001" />
@@ -41,5 +41,5 @@
       </inertial>
       <collision>
-        <origin xyz="0 0 0.0495" rpy="${pi} 0 ${-pi/2}" />
+        <origin xyz="0 0 0.0763" rpy="${pi} 0 ${-pi/2}" />
         <geometry>
           <mesh filename="file://$(find ${description_pkg})/urdf/meshes/avena/link_1.stl" scale="0.001 0.001 0.001" />
@@ -49,5 +49,5 @@
     <link name="${arm_id}_link_2">
       <visual>
-        <origin xyz="0 0 0.0495" rpy="0 ${pi} ${pi/2}" />
+        <origin xyz="0 0 0.0763" rpy="0 ${pi} ${pi/2}" />
         <geometry>
           <mesh filename="file://$(find ${description_pkg})/urdf/meshes/avena/link_2.stl" scale="0.001 0.001 0.001" />
@@ -61,5 +61,5 @@
       </inertial>
       <collision>
-        <origin xyz="0 0 0.0495" rpy="0 ${pi} ${pi/2}" />
+        <origin xyz="0 0 0.0763" rpy="0 ${pi} ${pi/2}" />
         <geometry>
           <mesh filename="file://$(find ${description_pkg})/urdf/meshes/avena/link_2.stl" scale="0.001 0.001 0.001" />
@@ -163,5 +163,5 @@
     </joint>
     <joint name="${arm_id}_joint_2" type="revolute">
-      <origin xyz="0.064 0 0.0495" rpy="0 ${pi/2} 0" />
+      <origin xyz="0.063 0 0.0763" rpy="0 ${pi/2} 0" />
       <parent link="${arm_id}_link_1" />
       <child link="${arm_id}_link_2" />
@@ -170,5 +170,5 @@
     </joint>
     <joint name="${arm_id}_joint_3" type="revolute">
-      <origin xyz="-0.452 0 0" rpy="0 ${pi} 0" />
+      <origin xyz="-0.467 0 0.009" rpy="0 ${pi} 0" />
       <parent link="${arm_id}_link_2" />
       <child link="${arm_id}_link_3" />

File: core/avena_bringup/urdf/avena_arm_ik_fast_new.urdf (robot description, URDF)
Before this commit: robot avena, 8 links, 7 joints
Joints:
- joint left_avena_joint_1: limit lower=-3.05 upper=3.05 effort=0 velocity=0 -> lower=-3.05 upper=3.05 effort=80 velocity=0
- joint left_avena_joint_2: limit lower=-1.57 upper=1.57 effort=0 velocity=0 -> lower=-1.57 upper=1.57 effort=180 velocity=0; origin xyz=0.064 0 0.0495 rpy=0 1.570796 0 -> xyz=0.063 0 0.0763 rpy=0 1.5708 0
- joint left_avena_joint_3: limit lower=-2.9 upper=2.9 effort=0 velocity=0 -> lower=-2.9 upper=2.9 effort=120 velocity=0; origin xyz=-0.452 0 0 rpy=0 3.141592 0 -> xyz=-0.467 0 0.009 rpy=0 3.1416 0
- joint left_avena_joint_4: limit lower=-3.05 upper=3.05 effort=0 velocity=0 -> lower=-3.05 upper=3.05 effort=60 velocity=0; origin xyz=0.452 0 0.0226 rpy=3.141592 0 0 -> xyz=0.452 0 0.0226 rpy=3.1416 0 0
- joint left_avena_joint_5: limit lower=-3.05 upper=3.05 effort=0 velocity=0 -> lower=-3.05 upper=3.05 effort=40 velocity=0; origin xyz=0.0495 0 0.064 rpy=0 -1.570796 3.141592 -> xyz=0.0495 0 0.064 rpy=0 -1.5708 3.1416
- joint left_avena_joint_6: limit lower=-3.05 upper=3.05 effort=0 velocity=0 -> lower=-3.05 upper=3.05 effort=40 velocity=0; origin xyz=0.0495 0 0.064 rpy=0 1.570796 0 -> xyz=0.0495 0 0.064 rpy=0 1.5708 0

Commit message: Add generated SRDF and YAML config files to workspace

File: core/avena_bringup/urdf/avena_arm.xacro (robot description, xacro)
@@ -6,5 +6,4 @@
   <xacro:macro name="avena_arm" params="arm_id:='avena' description_pkg:='avena_bringup'">
     <!-- Links -->
-    <link name="robot_base_link" />
     <link name="${arm_id}_link_0">
       <visual>
@@ -149,10 +148,4 @@
     <link name="${arm_id}_gripper_connection"/>
     <!-- Joints -->
-    <joint name="base_joint" type="fixed">
-      <origin rpy="0 0 0" xyz="0 0 0"/>
-      <parent link="robot_base_link"/>
-      <child link="${arm_id}_link_0"/>
-      <axis xyz="0 0 0"/>
-    </joint>
     <joint name="${arm_id}_joint_1" type="revolute">
       <origin xyz="0 0 0.063" rpy="0 0 -0.1963" /> <!-- Offset from position -->

Commit message: Add dummy "base_link" to URDF so KDL does not complain

File: core/avena_bringup/urdf/avena_arm.xacro (robot description, xacro)
@@ -6,4 +6,5 @@
   <xacro:macro name="avena_arm" params="arm_id:='avena' description_pkg:='avena_bringup'">
     <!-- Links -->
+    <link name="${arm_id}_base_link"/>
     <link name="${arm_id}_link_0">
       <visual>
@@ -148,4 +149,10 @@
     <link name="${arm_id}_gripper_connection"/>
     <!-- Joints -->
+    <joint name="${arm_id}_base_link_joint" type="fixed">
+      <origin xyz="0 0 0" rpy="0 0 0" />
+      <parent link="${arm_id}_base_link" />
+      <child link="${arm_id}_link_0" />
+      <axis xyz="0 0 0" />
+    </joint>
     <joint name="${arm_id}_joint_1" type="revolute">
       <origin xyz="0 0 0.063" rpy="0 0 -0.1963" /> <!-- Offset from position -->

Commit message: update urdf

File: core/avena_bringup/urdf/avena_arm.xacro (robot description, xacro)
@@ -37,5 +37,5 @@
       <inertial>
         <origin xyz="-0.00005 -0.007 0.0175 " rpy="0. 0. ${pi/2}"/>
-        <mass value="3.5"/>
+        <mass value="3.5+0.5"/>
         <inertia ixx="5.372e-03"  ixy="0."  ixz="0." iyy="4.691e-03" iyz="0." izz="5.059e-03" />
       </inertial>
@@ -56,6 +56,6 @@
       </visual>
       <inertial>
-        <origin xyz="0. 0.17651 0.01528" rpy="0. 0. ${pi/2}"/>
-        <mass value="6.3"/>
+        <origin xyz="-0.17651 0. 0.01528" rpy="0. ${pi} ${pi/2}"/>
+        <mass value="6.3+1"/>
         <inertia ixx="2.809e-01"  ixy="0."  ixz="0." iyy="8.463e-03" iyz="0." izz="2.804e-01" />
       </inertial>

Commit message: asdf

File: core/avena_bringup/urdf/avena_arm.xacro (robot description, xacro)
@@ -37,5 +37,5 @@
       <inertial>
         <origin xyz="-0.00005 -0.007 0.0175 " rpy="0. 0. ${pi/2}"/>
-        <mass value="3.5+0.5"/>
+        <mass value="3.8"/>
         <inertia ixx="5.372e-03"  ixy="0."  ixz="0." iyy="4.691e-03" iyz="0." izz="5.059e-03" />
       </inertial>
@@ -57,5 +57,5 @@
       <inertial>
         <origin xyz="-0.17651 0. 0.01528" rpy="0. ${pi} ${pi/2}"/>
-        <mass value="6.3+1"/>
+        <mass value="7."/>
         <inertia ixx="2.809e-01"  ixy="0."  ixz="0." iyy="8.463e-03" iyz="0." izz="2.804e-01" />
       </inertial>

Commit message: grav comp update

File: core/avena_bringup/urdf/avena_arm.xacro (robot description, xacro)
@@ -57,5 +57,5 @@
       <inertial>
         <origin xyz="-0.17651 0. 0.01528" rpy="0. ${pi} ${pi/2}"/>
-        <mass value="7."/>
+        <mass value="12."/>
         <inertia ixx="2.809e-01"  ixy="0."  ixz="0." iyy="8.463e-03" iyz="0." izz="2.804e-01" />
       </inertial>
@@ -77,5 +77,5 @@
       <inertial>
         <origin xyz="0.3046 0. 0.0588" rpy="0 0 ${pi/2}"/>
-        <mass value="3.375"/>
+        <mass value="2.4"/>
         <inertia ixx="1.149e-01"  ixy="0"  ixz="0" iyy="4.518e-03" iyz="0" izz="1.148e-01" />
       </inertial>

Commit message: param update

File: core/avena_bringup/urdf/avena_arm.xacro (robot description, xacro)
@@ -57,5 +57,5 @@
       <inertial>
         <origin xyz="-0.17651 0. 0.01528" rpy="0. ${pi} ${pi/2}"/>
-        <mass value="12."/>
+        <mass value="9."/>
         <inertia ixx="2.809e-01"  ixy="0."  ixz="0." iyy="8.463e-03" iyz="0." izz="2.804e-01" />
       </inertial>
@@ -77,5 +77,5 @@
       <inertial>
         <origin xyz="0.3046 0. 0.0588" rpy="0 0 ${pi/2}"/>
-        <mass value="2.4"/>
+        <mass value="3.375"/>
         <inertia ixx="1.149e-01"  ixy="0"  ixz="0" iyy="4.518e-03" iyz="0" izz="1.148e-01" />
       </inertial>

Commit message: long robot update

File: core/avena_bringup/urdf/avena_arm.xacro (robot description, xacro)
@@ -49,5 +49,5 @@
     <link name="${arm_id}_link_2">
       <visual>
-        <origin xyz="0 0 0.0763" rpy="0 ${pi} ${pi/2}" />
+        <origin xyz="0 0 0.0" rpy="0 ${pi} ${pi/2}" />
         <geometry>
           <mesh filename="file://$(find ${description_pkg})/urdf/meshes/avena/link_2.stl" scale="0.001 0.001 0.001" />
@@ -56,10 +56,10 @@
       </visual>
       <inertial>
-        <origin xyz="-0.17651 0. 0.01528" rpy="0. ${pi} ${pi/2}"/>
-        <mass value="9."/>
-        <inertia ixx="2.809e-01"  ixy="0."  ixz="0." iyy="8.463e-03" iyz="0." izz="2.804e-01" />
-      </inertial>
-      <collision>
-        <origin xyz="0 0 0.0763" rpy="0 ${pi} ${pi/2}" />
+        <origin xyz="-0.34301 0. -0.05751" rpy="0. ${pi} ${pi/2}"/>
+        <mass value="6.66"/>
+        <inertia ixx="6.3107e-01"  ixy="0."  ixz="0." iyy="9.544e-03" iyz="0." izz="6.301e-01" />
+      </inertial>
+      <collision>
+        <origin xyz="0 0 0" rpy="0 ${pi} ${pi/2}" />
         <geometry>
           <mesh filename="file://$(find ${description_pkg})/urdf/meshes/avena/link_2.stl" scale="0.001 0.001 0.001" />
@@ -69,5 +69,5 @@
     <link name="${arm_id}_link_3">
       <visual>
-        <origin xyz="0. 0. 0.0721" rpy="0 ${pi} ${-pi/2}" />
+        <origin xyz="0. 0. 0.0" rpy="0 ${pi} ${-pi/2}" />
         <geometry>
           <mesh filename="file://$(find ${description_pkg})/urdf/meshes/avena/link_3.stl" scale="0.001 0.001 0.001" />
@@ -76,10 +76,10 @@
       </visual>
       <inertial>
-        <origin xyz="0.3046 0. 0.0588" rpy="0 0 ${pi/2}"/>
-        <mass value="3.375"/>
-        <inertia ixx="1.149e-01"  ixy="0"  ixz="0" iyy="4.518e-03" iyz="0" izz="1.148e-01" />
-      </inertial>
-      <collision>
-        <origin xyz="0 0 0.0721" rpy="0 ${pi} ${-pi/2}" />
+        <origin xyz="0.3503 0. -0.051" rpy="0 0 ${pi/2}"/>
+        <mass value="3.666"/>
+        <inertia ixx="3.158e-01"  ixy="0"  ixz="0" iyy="6.297e-03" iyz="0" izz="3.160e-01" />
+      </inertial>
+      <collision>
+        <origin xyz="0 0 0" rpy="0 ${pi} ${-pi/2}" />
         <geometry>
           <mesh filename="file://$(find ${description_pkg})/urdf/meshes/avena/link_3.stl" scale="0.001 0.001 0.001" />
@@ -156,5 +156,5 @@
     </joint>
     <joint name="${arm_id}_joint_1" type="revolute">
-      <origin xyz="0 0 0.063" rpy="0 0 -0.1963" /> <!-- Offset from position -->
+      <origin xyz="0 0 0.063" rpy="0 0 0" /> <!-- Offset from position -->
       <parent link="${arm_id}_link_0" />
       <child link="${arm_id}_link_1" />
@@ -170,5 +170,5 @@
     </joint>
     <joint name="${arm_id}_joint_3" type="revolute">
-      <origin xyz="-0.467 0 0.009" rpy="0 ${pi} 0" />
+      <origin xyz="-0.686 0 0" rpy="0 ${pi} 0" />
       <parent link="${arm_id}_link_2" />
       <child link="${arm_id}_link_3" />
@@ -177,5 +177,5 @@
     </joint>
     <joint name="${arm_id}_joint_4" type="revolute">
-      <origin xyz="0.452 0 0.0226" rpy="${pi} 0 0" />
+      <origin xyz="0.671 0 -0.005" rpy="${pi} 0 0" />
       <parent link="${arm_id}_link_3" />
       <child link="${arm_id}_link_4" />

Commit message: params

File: core/avena_bringup/urdf/avena_arm.xacro (robot description, xacro)
@@ -56,7 +56,7 @@
       </visual>
       <inertial>
-        <origin xyz="-0.34301 0. -0.05751" rpy="0. ${pi} ${pi/2}"/>
-        <mass value="6.66"/>
-        <inertia ixx="6.3107e-01"  ixy="0."  ixz="0." iyy="9.544e-03" iyz="0." izz="6.301e-01" />
+        <origin xyz="-0.343 0. 0.05884" rpy="0. ${pi} ${pi/2}"/>
+        <mass value="9."/>
+        <inertia ixx="8.437e-01"  ixy="0."  ixz="0." iyy="1.143e-02" iyz="0." izz="8.428e-01" />
       </inertial>
       <collision>
@@ -76,7 +76,7 @@
       </visual>
       <inertial>
-        <origin xyz="0.3503 0. -0.051" rpy="0 0 ${pi/2}"/>
-        <mass value="3.666"/>
-        <inertia ixx="3.158e-01"  ixy="0"  ixz="0" iyy="6.297e-03" iyz="0" izz="3.160e-01" />
+        <origin xyz="0.38666 0. 0.051" rpy="0 0 ${pi/2}"/>
+        <mass value="5."/>
+        <inertia ixx="3.605e-01"  ixy="0"  ixz="0" iyy="6.825e-03" iyz="0" izz="3.606e-01" />
       </inertial>
       <collision>
@@ -97,5 +97,5 @@
       <inertial>
         <origin xyz="0.019 0. 0.059 " rpy="0. 0. ${pi/2}"/>
-        <mass value="1.960"/>
+        <mass value="2."/>
         <inertia ixx="2.233e-03"  ixy="0."  ixz="0." iyy="2.047e-03" iyz="0." izz="2.384e-03" />
       </inertial>
@@ -117,5 +117,5 @@
       <inertial>
         <origin xyz="0.019 0 0.059" rpy="0. 0. ${pi/2}"/>
-        <mass value="1.960"/>
+        <mass value="2."/>
         <inertia ixx="2.233e-03"  ixy="0."  ixz="0." iyy="2.047e-03" iyz="0." izz="2.384e-03" />
       </inertial>

Commit message: add velocity limit

File: core/avena_bringup/urdf/avena_arm.xacro (robot description, xacro)
@@ -160,5 +160,5 @@
       <child link="${arm_id}_link_1" />
       <axis xyz="0 0 1" />
-      <limit lower="-3.05" upper="3.05" effort="80" velocity="0" />
+      <limit lower="-3.05" upper="3.05" effort="80" velocity="1." />
     </joint>
     <joint name="${arm_id}_joint_2" type="revolute">
@@ -167,5 +167,5 @@
       <child link="${arm_id}_link_2" />
       <axis xyz="0 0 1" />
-      <limit lower="-1.57" upper="1.57" effort="180" velocity="0" />
+      <limit lower="-1.57" upper="1.57" effort="200" velocity="1." />
     </joint>
     <joint name="${arm_id}_joint_3" type="revolute">
@@ -174,5 +174,5 @@
       <child link="${arm_id}_link_3" />
       <axis xyz="0 0 1" />
-      <limit lower="-2.9" upper="2.9" effort="120" velocity="0" />
+      <limit lower="-2.9" upper="2.9" effort="120" velocity="1." />
     </joint>
     <joint name="${arm_id}_joint_4" type="revolute">
@@ -181,5 +181,5 @@
       <child link="${arm_id}_link_4" />
       <axis xyz="0 0 1" />
-      <limit lower="-3.05" upper="3.05" effort="60" velocity="0" />
+      <limit lower="-3.05" upper="3.05" effort="60" velocity="1." />
     </joint>
     <joint name="${arm_id}_joint_5" type="revolute">
@@ -188,5 +188,5 @@
       <child link="${arm_id}_link_5" />
       <axis xyz="0 0 1" />
-      <limit lower="-3.05" upper="3.05" effort="40" velocity="0" />
+      <limit lower="-3.05" upper="3.05" effort="40" velocity="1." />
     </joint>
     <joint name="${arm_id}_joint_6" type="revolute">
@@ -195,5 +195,5 @@
       <child link="${arm_id}_link_6" />
       <axis xyz="0 0 1" />
-      <limit lower="-3.05" upper="3.05" effort="40" velocity="0" />
+      <limit lower="-3.05" upper="3.05" effort="40" velocity="1." />
     </joint>
     <joint name="${arm_id}_joint_7" type="fixed">

Commit message: fix stuff

File: core/avena_bringup/urdf/avena_arm.xacro (robot description, xacro)
@@ -203,4 +203,4 @@
       <axis xyz="0 0 0" />
     </joint>
- </xacro:macro>
+  </xacro:macro>
 </robot>
