Commit message: Resolve "Spawn collision items"

File: core/avena_bringup/worlds/avena_table.xacro (robot description, xacro)
@@ -6,19 +6,26 @@
   </material>
   <!-- Collision box -->
-  <xacro:macro name="collision_box" params="name size transparent:='false' xyz:='0 0 0' rpy:='0 0 0' base_link:='base_link'">
+  <xacro:macro name="collision_box" params="name size visual:='true' transparent:='false' xyz:='0 0 0' rpy:='0 0 0' rgba:='0.8 0.8 0.8 1' table_base_link:='table_base_link'">
     <joint name="${name}" type="fixed">
       <origin xyz="${xyz}" rpy="${rpy}" />
-      <parent link="${base_link}" />
+      <parent link="${table_base_link}" />
       <child link="${name}" />
     </joint>
     <link name="${name}">
-      <visual>
-        <geometry>
-          <box size="${size}"/>
-        </geometry>
-        <xacro:if value="${transparent}">
-          <material name="transparent" />
-        </xacro:if>
-      </visual>
+      <xacro:if value="${visual}">
+        <visual>
+          <geometry>
+            <box size="${size}"/>
+          </geometry>
+          <xacro:if value="${transparent}">
+            <material name="transparent" />
+          </xacro:if>
+          <xacro:unless value="${transparent}">
+            <material name="custom_color">
+              <color rgba="${rgba}" />
+            </material>
+          </xacro:unless>
+        </visual>
+      </xacro:if>
       <collision>
         <geometry>
@@ -40,5 +47,5 @@
     <xacro:property name="camera_size" value="0.1" />
     <xacro:property name="camera_height" value="1.05" />
-    <link name="base_link"/>
+    <link name="table_base_link"/>
     <!-- Table top -->
     <xacro:collision_box
@@ -46,4 +53,5 @@
       xyz="${x_origin} ${y_origin} ${-thickness / 2}"
       size="${x_dim} ${y_dim} ${thickness}"
+      rgba="1 0.6 0.5 1"
     />
     <!-- ********************************************* -->
@@ -54,4 +62,5 @@
       size="${thickness} ${y_dim} ${walls_height}"
       transparent="true"
+      visual="false"
     />
     <xacro:collision_box

Commit message: Update scene description

File: core/avena_bringup/worlds/avena_table.xacro (robot description, xacro)
@@ -28,4 +28,5 @@
  <!-- Table -->
   <xacro:macro name="table" params="x_min:=0 x_max:=0 y_min:=0 y_max:=0">
+    <!-- When physical scene changes, check dimensions of static objects -->
     <xacro:property name="wall_thickness" value="0.01" />
     <xacro:property name="walls_height" value="1.7" />
@@ -34,8 +35,11 @@
     <xacro:property name="x_dim" value="${x_max - x_min}" />
     <xacro:property name="y_dim" value="${y_max - y_min}" />
-    <xacro:property name="stick_size" value="0.05" />
-    <xacro:property name="stick_height" value="${walls_height}" />
-    <xacro:property name="camera_size" value="0.1" />
-    <xacro:property name="camera_height" value="1.05" />
+    <xacro:property name="column_size" value="0.05" />
+    <xacro:property name="column_height" value="${walls_height}" />
+    <xacro:property name="camera_dim_x" value="0.12" />
+    <xacro:property name="camera_dim_y" value="0.2" />
+    <xacro:property name="camera_dim_z" value="0.2" />
+    <xacro:property name="camera_height" value="0.72" />
+    <xacro:property name="column_pos_offset" value="0.8" />
     <link name="table_base_link"/>
     <!-- Table top -->
@@ -73,65 +77,73 @@
     />
     <xacro:collision_box
-      name="temp_left_collision_wall_0"
-      xyz="${x_dim / 2} 0.7 ${walls_height / 2}"
-      size="${x_dim} ${wall_thickness} ${walls_height}"
-      rgba="1 1 1 0.2"
-    />
-    <xacro:collision_box
-      name="temp_left_collision_wall_1"
-      xyz="${x_dim / 2} 0.1 ${walls_height / 2}"
+      name="temp_collision_wall_0"
+      xyz="${x_dim / 2} -0.3 ${walls_height / 2}"
       size="${x_dim} ${wall_thickness} ${walls_height}"
       rgba="1 1 1 0.2"
     />
     <!-- ********************************************* -->
-    <!-- STICKS -->
+    <!-- COLUMN -->
     <xacro:collision_box
-      name="left_back"
-      xyz="${stick_size / 2} 0.8 ${stick_height / 2}"
-      size="${stick_size} ${2 * stick_size} ${stick_height}"
+      name="left_back_column"
+      xyz="${column_size / 2} ${column_pos_offset} ${column_height / 2}"
+      size="${column_size} ${2 * column_size} ${column_height}"
       visual="false"
     />
     <xacro:collision_box
-      name="left_front"
-      xyz="${x_dim - stick_size / 2} 0.8 ${stick_height / 2}"
-      size="${stick_size} ${2 * stick_size} ${stick_height}"
+      name="left_front_column"
+      xyz="${x_dim - column_size / 2} ${column_pos_offset} ${column_height / 2}"
+      size="${column_size} ${2 * column_size} ${column_height}"
       visual="false"
     />
     <xacro:collision_box
-      name="middle_front"
-      xyz="${x_dim - stick_size / 2} 0 ${stick_height / 2}"
-      size="${stick_size} ${2 * stick_size} ${stick_height}"
+      name="middle_front_column"
+      xyz="${x_dim - column_size / 2} 0 ${column_height / 2}"
+      size="${column_size} ${2 * column_size} ${column_height}"
       visual="false"
     />
     <xacro:collision_box
-      name="middle_back"
-      xyz="${stick_size / 2} 0 ${stick_height / 2}"
-      size="${stick_size} ${2 * stick_size} ${stick_height}"
+      name="middle_back_column"
+      xyz="${column_size / 2} 0 ${column_height / 2}"
+      size="${column_size} ${2 * column_size} ${column_height}"
       visual="false"
     />
     <xacro:collision_box
-      name="right_front"
-      xyz="${x_dim - stick_size / 2} -0.8 ${stick_height / 2}"
-      size="${stick_size} ${2 * stick_size} ${stick_height}"
+      name="right_front_column"
+      xyz="${x_dim - column_size / 2} ${-column_pos_offset} ${column_height / 2}"
+      size="${column_size} ${2 * column_size} ${column_height}"
       visual="false"
     />
     <xacro:collision_box
-      name="right_back"
-      xyz="${stick_size / 2} -0.8 ${stick_height / 2}"
-      size="${stick_size} ${2 * stick_size} ${stick_height}"
+      name="right_back_column"
+      xyz="${column_size / 2} ${-column_pos_offset} ${column_height / 2}"
+      size="${column_size} ${2 * column_size} ${column_height}"
       visual="false"
     />
     <!-- ********************************************* -->
     <!-- CAMERAS -->
-    <!-- <xacro:collision_box
-      name="left_camera"
-      xyz="${x_max - camera_size / 2} ${y_max - camera_size / 2} ${camera_height}"
-      size="${camera_size} ${camera_size} ${camera_size}"
-    /> -->
-    <!-- <xacro:collision_box
-      name="right_camera"
-      xyz="${x_max - camera_size / 2} ${y_min + camera_size / 2} ${camera_height}"
-      size="${camera_size} ${camera_size} ${camera_size}"
-    /> -->
+    <xacro:collision_box
+      name="left_back_camera"
+      xyz="${camera_dim_x / 2} ${column_pos_offset} ${camera_height}"
+      size="${camera_dim_x} ${camera_dim_y} ${camera_dim_z}"
+      visual="false"
+    />
+    <xacro:collision_box
+      name="left_front_camera"
+      xyz="${x_dim - camera_dim_x / 2} ${column_pos_offset} ${camera_height}"
+      size="${camera_dim_x} ${camera_dim_y} ${camera_dim_z}"
+      visual="false"
+    />
+    <xacro:collision_box
+      name="middle_back_camera"
+      xyz="${camera_dim_x / 2} 0 ${camera_height}"
+      size="${camera_dim_x} ${camera_dim_y} ${camera_dim_z}"
+      visual="false"
+    />
+    <xacro:collision_box
+      name="middle_front_camera"
+      xyz="${x_dim - camera_dim_x / 2} 0 ${camera_height}"
+      size="${camera_dim_x} ${camera_dim_y} ${camera_dim_z}"
+      visual="false"
+    />
   </xacro:macro>
 </robot>

Commit message: asdf

File: core/avena_bringup/worlds/avena_table.xacro (robot description, xacro)
@@ -37,4 +37,5 @@
     <xacro:property name="column_size" value="0.05" />
     <xacro:property name="column_height" value="${walls_height}" />
+    <xacro:property name="bar_height" value="1." />
     <xacro:property name="camera_dim_x" value="0.12" />
     <xacro:property name="camera_dim_y" value="0.2" />
@@ -97,4 +98,10 @@
     />
     <xacro:collision_box
+      name="left_bar"
+      xyz="${x_dim / 2} ${column_pos_offset} ${bar_height}"
+      size="${x_dim} ${2 * column_size} ${column_size}"
+      visual="false"
+    />
+    <xacro:collision_box
       name="middle_front_column"
       xyz="${x_dim - column_size / 2} 0 ${column_height / 2}"
